File: board/PlantCtrlESP32.kicad_pcb (KiCad board)
At the start: 2 copper layers, 99.1 x 99.1 mm, 140 parts, among them IC1 DW01, J1 Conn_01x03_Female, J2 Conn_01x04, J3 Conn_01x04, J4 Conn_01x02_Female, J5 Conn_01x04, J6 Conn_01x03, J7 Conn_01x02, Q1 SL2300, Q10 SL2300, Q11 SL2300, Q12 SL2300, Q2 SL2300, Q3 SL2300, Q4 SL2300, Q5 SL2300, Q6 SL2300, Q7 SL2300, Q8 SL2300, Q9 SL2300, U1 DS18B20, U2 ESP32-DEVKITC-32D, U3 LP38690DT-3.3, U4 SX1308

Commit message: fixed wrong mosefets used
Other:
- board text added: "PlantCtrl V0.5"
- board text removed: "PlantCtrl V0.4"

Commit message: updated pcb
Parts:
- D8: value B0520LW -> 40V 1A
- Pumps1: value LED -> LED_red
- Q1, Q10, Q11, Q12, Q2, Q3, Q4, Q5, Q6, Q7, Q8, Q9: value SL2300 -> N-channel 30V 5A
- Q_PWR1, Q_PWR2: value BSS84 -> P-channel 50v 4A
- R11, R13, R15, R18, R30, R31, R5, R7, R9: value 255 -> 270
- R21: value 14-19k -> 18k
- Sensor1: value LED -> LED_green
Changed lines of the file:
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@@
     (add_net "Net-(Hall1-Pad3)")
     (add_net "Net-(IC1-Pad2)")
+    (add_net "Net-(IC1-Pad4)")
     (add_net "Net-(J5-Pad2)")
     (add_net "Net-(J5-Pad3)")
@@
     (add_net "Net-(R45-Pad1)")
     (add_net "Net-(R49-Pad1)")
+    (add_net "Net-(U2-Pad16)")
+    (add_net "Net-(U2-Pad17)")
+    (add_net "Net-(U2-Pad18)")
+    (add_net "Net-(U2-Pad19)")
+    (add_net "Net-(U2-Pad2)")
+    (add_net "Net-(U2-Pad3)")
+    (add_net "Net-(U2-Pad33)")
+    (add_net "Net-(U2-Pad36)")
+    (add_net "Net-(U2-Pad37)")
+    (add_net "Net-(U2-Pad38)")
+    (add_net "Net-(U2-Pad4)")
+    (add_net "Net-(U4-Pad6)")
     (add_net PLANT0_MOIST)
     (add_net PLANT0_PUMP)
@@
       (effects (font (size 1 1) (thickness 0.15)))
     )
-    (fp_text value LED (at 0 1.65 90) (layer F.Fab)
+    (fp_text value LED_green (at 0 1.65 90) (layer F.Fab)
       (effects (font (size 1 1) (thickness 0.15)))
     )
@@
       (effects (font (size 1 1) (thickness 0.15)))
     )
-    (fp_text value LED (at 0 1.65 90) (layer F.Fab)
+    (fp_text value LED_red (at 0 1.65 90) (layer F.Fab)
       (effects (font (size 1 1) (thickness 0.15)))
     )
@@
       (effects (font (size 1 1) (thickness 0.15)))
     )
-    (fp_text value 255 (at 0 1.65 90) (layer F.Fab)
+    (fp_text value 270 (at 0 1.65 90) (layer F.Fab)
       (effects (font (size 1 1) (thickness 0.15)))
     )
@@
       (effects (font (size 1 1) (thickness 0.15)))
     )
-    (fp_text value 255 (at 0 1.65 90) (layer F.Fab)
+    (fp_text value 270 (at 0 1.65 90) (layer F.Fab)
       (effects (font (size 1 1) (thickness 0.15)))
     )
@@
       (effects (font (size 1 1) (thickness 0.15)))
     )
-    (fp_text value 255 (at 0 1.65 90) (layer F.Fab)
+    (fp_text value 270 (at 0 1.65 90) (layer F.Fab)
       (effects (font (size 1 1) (thickness 0.15)))
     )
@@
       (effects (font (size 1 1) (thickness 0.15)))
     )
-    (fp_text value 255 (at 0 1.65 90) (layer F.Fab)
+    (fp_text value 270 (at 0 1.65 90) (layer F.Fab)
       (effects (font (size 1 1) (thickness 0.15)))
     )
@@
       (effects (font (size 1 1) (thickness 0.15)))
     )
-    (fp_text value 255 (at 0 1.65 90) (layer F.Fab)
+    (fp_text value 270 (at 0 1.65 90) (layer F.Fab)
       (effects (font (size 1 1) (thickness 0.15)))
     )
@@
       (effects (font (size 1 1) (thickness 0.15)))
     )
-    (fp_text value 255 (at 0 1.65 90) (layer F.Fab)
+    (fp_text value 270 (at 0 1.65 90) (layer F.Fab)
       (effects (font (size 1 1) (thickness 0.15)))
     )
@@
       (effects (font (size 1 1) (thickness 0.15)))
     )
-    (fp_text value 255 (at 0 1.65 90) (layer F.Fab)
+    (fp_text value 270 (at 0 1.65 90) (layer F.Fab)
       (effects (font (size 1 1) (thickness 0.15)))
     )
@@
       (effects (font (size 1 1) (thickness 0.15)))
     )
-    (fp_text value 255 (at 0 1.65 90) (layer F.Fab)
+    (fp_text value 270 (at 0 1.65 90) (layer F.Fab)
       (effects (font (size 1 1) (thickness 0.15)))
     )
@@
       (effects (font (size 1 1) (thickness 0.15)))
     )
-    (fp_text value 255 (at 0 1.65 90) (layer F.Fab)
+    (fp_text value 270 (at 0 1.65 90) (layer F.Fab)
       (effects (font (size 1 1) (thickness 0.15)))
     )
@@
       (effects (font (size 1 1) (thickness 0.15)))
     )
-    (fp_text value BSS84 (at 0 2.5 90) (layer F.Fab)
+    (fp_text value "P-channel 50v 4A" (at 0 2.5 90) (layer F.Fab)
       (effects (font (size 1 1) (thickness 0.15)))
     )
@@
       (effects (font (size 1 1) (thickness 0.15)))
     )
-    (fp_text value BSS84 (at 0 2.54 90) (layer F.Fab)
+    (fp_text value "P-channel 50v 4A" (at 0 2.54 90) (layer F.Fab)
       (effects (font (size 1 1) (thickness 0.15)))
     )
@@
       (effects (font (size 1 1) (thickness 0.15)))
     )
-    (fp_text value SL2300 (at 0 2.5 90) (layer F.Fab)
+    (fp_text value "N-channel 30V 5A" (at 0 2.5 90) (layer F.Fab)
       (effects (font (size 1 1) (thickness 0.15)))
     )
@@
       (effects (font (size 1 1) (thickness 0.15)))
     )
-    (fp_text value SL2300 (at 0 2.5 90) (layer F.Fab)
+    (fp_text value "N-channel 30V 5A" (at 0 2.5 90) (layer F.Fab)
       (effects (font (size 1 1) (thickness 0.15)))
     )
@@
       (effects (font (size 1 1) (thickness 0.15)))
     )
-    (fp_text value SL2300 (at 0 2.5 90) (layer F.Fab)
+    (fp_text value "N-channel 30V 5A" (at 0 2.5 90) (layer F.Fab)
       (effects (font (size 1 1) (thickness 0.15)))
     )
@@
       (effects (font (size 1 1) (thickness 0.15)))
     )
-    (fp_text value SL2300 (at 0 2.5 90) (layer F.Fab)
+    (fp_text value "N-channel 30V 5A" (at 0 2.5 90) (layer F.Fab)
       (effects (font (size 1 1) (thickness 0.15)))
     )
@@
       (effects (font (size 1 1) (thickness 0.15)))
     )
-    (fp_text value SL2300 (at 0 2.5) (layer F.Fab)
+    (fp_text value "N-channel 30V 5A" (at 0 2.5) (layer F.Fab)
       (effects (font (size 1 1) (thickness 0.15)))
     )
@@
       (effects (font (size 1 1) (thickness 0.15)))
     )
-    (fp_text value SL2300 (at 0 2.5 90) (layer F.Fab)
+    (fp_text value "N-channel 30V 5A" (at 0 2.5 90) (layer F.Fab)
       (effects (font (size 1 1) (thickness 0.15)))
     )
@@
       (effects (font (size 1 1) (thickness 0.15)))
     )
-    (fp_text value SL2300 (at 0 2.5 90) (layer F.Fab)
+    (fp_text value "N-channel 30V 5A" (at 0 2.5 90) (layer F.Fab)
       (effects (font (size 1 1) (thickness 0.15)))
     )
@@
       (effects (font (size 1 1) (thickness 0.15)))
     )
-    (fp_text value SL2300 (at 0 2.5 90) (layer F.Fab)
+    (fp_text value "N-channel 30V 5A" (at 0 2.5 90) (layer F.Fab)
       (effects (font (size 1 1) (thickness 0.15)))
     )
@@
       (effects (font (size 1 1) (thickness 0.15)))
     )
-    (fp_text value SL2300 (at 0 2.5 90) (layer F.Fab)
+    (fp_text value "N-channel 30V 5A" (at 0 2.5 90) (layer F.Fab)
       (effects (font (size 1 1) (thickness 0.15)))
     )
@@
       (effects (font (size 1 1) (thickness 0.15)))
     )
-    (fp_text value SL2300 (at 0 2.5 90) (layer F.Fab)
+    (fp_text value "N-channel 30V 5A" (at 0 2.5 90) (layer F.Fab)
       (effects (font (size 1 1) (thickness 0.15)))
     )
@@
       (effects (font (size 1 1) (thickness 0.15)))
     )
-    (fp_text value 14-19k (at 0 1.65 90) (layer F.Fab)
+    (fp_text value 18k (at 0 1.65 90) (layer F.Fab)
       (effects (font (size 1 1) (thickness 0.15)))
     )
@@
       (effects (font (size 1 1) (thickness 0.15)))
     )
-    (fp_text value B0520LW (at 0 2.1) (layer F.Fab)
+    (fp_text value "40V 1A" (at 0 2.1) (layer F.Fab)
       (effects (font (size 1 1) (thickness 0.15)))
     )
@@
       (effects (font (size 1 1) (thickness 0.15)))
     )
-    (fp_text value SL2300 (at 0 2.5 90) (layer F.Fab)
+    (fp_text value "N-channel 30V 5A" (at 0 2.5 90) (layer F.Fab)
       (effects (font (size 1 1) (thickness 0.15)))
     )
@@
       (effects (font (size 1 1) (thickness 0.15)))
     )
-    (fp_text value SL2300 (at 0 2.5 90) (layer F.Fab)
+    (fp_text value "N-channel 30V 5A" (at 0 2.5 90) (layer F.Fab)
       (effects (font (size 1 1) (thickness 0.15)))
     )

Commit message: Added capacitor for ESP
Parts:
- added C14: 100u, Capacitor_THT:CP_Radial_D12.5mm_P5.00mm, F.Cu at (217.2, 85.2)
Routing:
- net 3_3V: track 154.5 -> 197.5 mm, vias 4 -> 6
- net Net-(C1-Pad2): track 116.7 -> 120.9 mm

Commit message: Moved J6 under lipo
Parts:
- moved JP6 25.9 mm to (210.4, 63.6), turned to 180 degrees
Routing:
- net 3_3V: track 197.5 -> 206.2 mm
- net LIPO+: track 301.0 -> 301.8 mm
Changed lines of the file:
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@@
     (thickness 1.6)
     (drawings 10)
-    (tracks 891)
+    (tracks 895)
     (zones 0)
     (modules 141)
@@
   )
   (module Jumper:SolderJumper-2_P1.3mm_Open_Pad1.0x1.5mm (layer F.Cu)
-    (at 191.77 81.534)
+    (at 210.4136 63.5508 180)
     (descr "SMD Solder Jumper, 1x1.5mm Pads, 0.3mm gap, open")
     (tags "solder jumper open")
@@
     (fp_line (start 1.65 1.25) (end 1.65 -1.25) (layer F.CrtYd) (width 0.05))
     (fp_line (start 1.65 1.25) (end -1.65 1.25) (layer F.CrtYd) (width 0.05))
-    (pad 1 smd rect (at -0.65 0) (size 1 1.5) (layers F.Cu F.Mask)
+    (pad 1 smd rect (at -0.65 0 180) (size 1 1.5) (layers F.Cu F.Mask)
       (net 20 3_3V))
-    (pad 2 smd rect (at 0.65 0) (size 1 1.5) (layers F.Cu F.Mask)
+    (pad 2 smd rect (at 0.65 0 180) (size 1 1.5) (layers F.Cu F.Mask)
       (net 15 LIPO+))
   )
@@
   (segment (start 252.73 82.55) (end 252.73 81.534) (width 1.2) (layer F.Cu) (net 15) (status 30))
   (segment (start 248.158 87.122) (end 252.73 82.55) (width 1.2) (layer F.Cu) (net 15) (status 20))
-  (segment (start 193.547 78.364) (end 193.547 79.674) (width 0.2) (layer F.Cu) (net 15) (status 10))
-  (segment (start 192.42 79.491) (end 193.547 78.364) (width 1) (layer F.Cu) (net 15) (status 20))
-  (segment (start 192.42 81.534) (end 192.42 79.491) (width 1) (layer F.Cu) (net 15) (status 10))
-  (segment (start 192.42 82.076) (end 192.42 81.534) (width 0.2) (layer F.Cu) (net 15) (status 30))
-  (segment (start 189.676 84.82) (end 192.42 82.076) (width 0.2) (layer F.Cu) (net 15) (status 20))
-  (segment (start 188.976 84.82) (end 189.676 84.82) (width 0.2) (layer F.Cu) (net 15) (status 10))
   (segment (start 194.441 77.47) (end 193.547 78.364) (width 1) (layer F.Cu) (net 15) (status 20))
   (segment (start 200.914 72.39) (end 200.533 72.771) (width 1) (layer B.Cu) (net 15))
@@
   (segment (start 199.2122 72.771) (end 200.533 72.771) (width 1) (layer F.Cu) (net 15))
   (segment (start 194.5132 77.47) (end 199.2122 72.771) (width 1) (layer F.Cu) (net 15))
+  (segment (start 189.676 84.82) (end 188.976 84.82) (width 0.2) (layer F.Cu) (net 15))
+  (segment (start 193.5988 80.8972) (end 189.676 84.82) (width 0.2) (layer F.Cu) (net 15))
+  (segment (start 193.5988 79.6036) (end 193.5988 80.8972) (width 0.2) (layer F.Cu) (net 15))
+  (segment (start 193.547 78.364) (end 193.5988 79.6036) (width 0.2) (layer F.Cu) (net 15))
+  (segment (start 208.2904 65.024) (end 209.7636 63.5508) (width 1.2) (layer F.Cu) (net 15))
+  (segment (start 208.28 65.024) (end 208.2904 65.024) (width 1.2) (layer F.Cu) (net 15))
   (segment (start 260.588 79.74) (end 259.842 78.994) (width 0.2) (layer F.Cu) (net 16) (status 20))
   (segment (start 265.938 79.74) (end 260.588 79.74) (width 0.2) (layer F.Cu) (net 16) (status 10))
@@
   (segment (start 192.278 82.692) (end 189.794 80.208) (width 0.2) (layer B.Cu) (net 20))
   (segment (start 192.278 88.9) (end 192.278 82.692) (width 0.2) (layer B.Cu) (net 20))
-  (segment (start 189.794 80.208) (end 191.12 81.534) (width 1) (layer F.Cu) (net 20) (status 20))
   (segment (start 188.977 79.391) (end 189.794 80.208) (width 1) (layer F.Cu) (net 20) (status 10))
   (via (at 192.024 99.822) (size 0.8) (drill 0.4) (layers F.Cu B.Cu) (net 20))
@@
   (segment (start 188.977 77.48) (end 186.182 74.685) (width 1.2) (layer F.Cu) (net 20) (status 30))
   (segment (start 188.977 78.364) (end 188.977 77.48) (width 1.2) (layer F.Cu) (net 20) (status 30))
-  (segment (start 217.2208 85.1916) (end 215.7984 83.7692) (width 1) (layer B.Cu) (net 20))
-  (segment (start 215.7984 83.7692) (end 210.6676 83.7692) (width 1) (layer B.Cu) (net 20))
-  (segment (start 210.6676 83.7692) (end 210.2104 83.7692) (width 1) (layer B.Cu) (net 20))
-  (segment (start 210.2104 83.7692) (end 209.0928 82.6516) (width 1) (layer B.Cu) (net 20))
-  (segment (start 209.0928 82.6516) (end 209.0928 74.5236) (width 1) (layer B.Cu) (net 20))
-  (segment (start 209.0928 74.5236) (end 206.7052 72.136) (width 1) (layer B.Cu) (net 20))
-  (segment (start 203.00649 72.136) (end 198.4756 76.66689) (width 1) (layer B.Cu) (net 20))
-  (segment (start 206.7052 72.136) (end 203.00649 72.136) (width 1) (layer B.Cu) (net 20))
-  (via (at 198.4756 76.66689) (size 0.8) (drill 0.4) (layers F.Cu B.Cu) (net 20))
   (segment (start 189.794 80.208) (end 198.3688 80.208) (width 1) (layer B.Cu) (net 20))
   (via (at 198.3688 80.208) (size 0.8) (drill 0.4) (layers F.Cu B.Cu) (net 20))
   (segment (start 198.4756 80.1012) (end 198.3688 80.208) (width 1) (layer F.Cu) (net 20))
   (segment (start 198.4756 76.66689) (end 198.4756 80.1012) (width 1) (layer F.Cu) (net 20))
+  (segment (start 211.0636 65.3008) (end 207.1624 69.202) (width 1) (layer F.Cu) (net 20))
+  (segment (start 211.0636 63.5508) (end 211.0636 65.3008) (width 1) (layer F.Cu) (net 20))
+  (segment (start 207.1624 69.202) (end 207.1624 72.644) (width 1) (layer F.Cu) (net 20))
+  (via (at 207.1624 72.644) (size 0.8) (drill 0.4) (layers F.Cu B.Cu) (net 20))
+  (segment (start 210.2104 83.7692) (end 215.7984 83.7692) (width 1) (layer B.Cu) (net 20))
+  (segment (start 209.0928 82.6516) (end 210.2104 83.7692) (width 1) (layer B.Cu) (net 20))
+  (segment (start 215.7984 83.7692) (end 217.2208 85.1916) (width 1) (layer B.Cu) (net 20))
+  (segment (start 209.0928 74.5236) (end 209.0928 82.6516) (width 1) (layer B.Cu) (net 20))
+  (segment (start 207.613199 73.043999) (end 209.0928 74.5236) (width 1) (layer B.Cu) (net 20))
+  (segment (start 207.562399 73.043999) (end 207.613199 73.043999) (width 1) (layer B.Cu) (net 20))
+  (segment (start 207.1624 72.644) (end 207.562399 73.043999) (width 1) (layer B.Cu) (net 20))
+  (segment (start 202.898489 72.244001) (end 198.4756 76.66689) (width 1) (layer F.Cu) (net 20))
+  (segment (start 206.762401 72.244001) (end 202.898489 72.244001) (width 1) (layer F.Cu) (net 20))
+  (segment (start 207.1624 72.644) (end 206.762401 72.244001) (width 1) (layer F.Cu) (net 20))
   (via (at 201.93 127) (size 0.8) (drill 0.4) (layers F.Cu B.Cu) (net 21))
   (segment (start 203.47 127) (end 201.93 127) (width 0.2) (layer F.Cu) (net 21) (status 10))

Commit message: Removed deadend wires at S6
Routing:
- net GND: track 781.7 -> 766.3 mm
- net PWR_SENSORS: track 247.8 -> 243.6 mm
Changed lines of the file:
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@@
     (thickness 1.6)
     (drawings 10)
-    (tracks 895)
+    (tracks 889)
     (zones 0)
     (modules 141)
@@
   )
   (setup
-    (last_trace_width 1)
+    (last_trace_width 1.2)
     (user_trace_width 0.2)
     (user_trace_width 0.5)
@@
   (segment (start 212.486 131.684) (end 214.63 129.54) (width 0.2) (layer F.Cu) (net 7) (status 20))
   (segment (start 211.328 131.684) (end 212.486 131.684) (width 0.2) (layer F.Cu) (net 7) (status 10))
-  (segment (start 259.478676 118.96699) (end 259.07499 119.370676) (width 0.2) (layer F.Cu) (net 7))
-  (segment (start 259.07499 119.370676) (end 259.07499 128.26499) (width 0.2) (layer F.Cu) (net 7))
-  (segment (start 261.96899 118.96699) (end 259.478676 118.96699) (width 0.2) (layer F.Cu) (net 7))
-  (segment (start 259.07499 128.26499) (end 260.35 129.54) (width 0.2) (layer F.Cu) (net 7) (status 20))
-  (segment (start 263.144 120.142) (end 261.96899 118.96699) (width 0.2) (layer F.Cu) (net 7))
   (segment (start 185.42 118.5965) (end 199.136 118.5965) (width 0.2) (layer F.Cu) (net 7) (status 30))
   (segment (start 173.788 113.792) (end 179.705 107.875) (width 0.2) (layer F.Cu) (net 7) (status 30))
@@
   (segment (start 260.35 124.54) (end 214.63 124.54) (width 0.2) (layer B.Cu) (net 24) (status 30))
   (segment (start 260.169 124.359) (end 260.35 124.54) (width 0.2) (layer F.Cu) (net 24) (status 30))
-  (segment (start 260.169 120.142) (end 260.169 124.359) (width 0.2) (layer F.Cu) (net 24) (status 20))
   (segment (start 173.736 121.666) (end 186.055 133.985) (width 0.2) (layer F.Cu) (net 24) (status 20))
   (segment (start 173.736 118.792) (end 173.736 121.666) (width 0.2) (layer F.Cu) (net 24) (status 10))
@@
     (connect_pads (clearance 0.508))
     (min_thickness 0.254)
-    (fill (arc_segments 32) (thermal_gap 0.508) (thermal_bridge_width 0.508))
+    (fill yes (arc_segments 32) (thermal_gap 0.508) (thermal_bridge_width 0.508))
     (polygon
       (pts
@@
     (connect_pads (clearance 0.508))
     (min_thickness 0.254)
-    (fill (arc_segments 32) (thermal_gap 0.508) (thermal_bridge_width 0.508))
+    (fill yes (arc_segments 32) (thermal_gap 0.508) (thermal_bridge_width 0.508))
     (polygon
       (pts

Commit message: Added J8 for USB programming and POWER supply by USB; Lipo has to be disconnected!
Parts:
- added D26: 40V >2A, Diode_SMD:D_SOD-123F, F.Cu at (248.1, 72.1)
- added J8: Conn_01x02, Connector_PinHeader_2.54mm:PinHeader_2x01_P2.54mm_Vertical, F.Cu at (177.1, 124.0)
- D8: value 40V 1A -> 40V >2A
- L1: value LQH32CN100K33L -> 4A 5-22uH min DCR
- R21: value 18k -> 19k-19.5K
- moved R21 0.61 mm to (245.8, 72.1)
- moved R29 0.61 mm to (243.5, 72.1)
Connections:
- C12 pad 1: PUMP_PWR -> Net-(C12-Pad1)
- D8 pad 1: PUMP_PWR -> Net-(C12-Pad1)
- R21 pad 1: PUMP_PWR -> Net-(C12-Pad1)
- U2 pad 19: (no net) -> EXT_5V
Routing:
- net LIPO+: track 301.8 -> 341.4 mm, vias 10 -> 11
- net PUMP_PWR: track 195.0 -> 184.3 mm
- net Net-(C12-Pad1): track 0.00 -> 8.09 mm
- net PWR_SENSORS: track 243.6 -> 250.4 mm
- net EXT_5V: track 0.00 -> 3.46 mm
- net GND: track 766.3 -> 763.2 mm
- net Temp: track 143.1 -> 145.5 mm
- net Net-(J5-Pad2): track 12.8 -> 14.3 mm
- net Net-(R21-Pad2): track 6.96 -> 6.26 mm
