File: board/PlantCtrlESP32.kicad_pcb (KiCad board)
At the start: 2 copper layers, 99.1 x 99.1 mm, 170 parts, among them IC1 DW01, J1 Conn_01x06_Female, Q1 N-channel 30V 5A, Q10 N-channel 30V 5A, Q11 N-channel 30V 5A, Q12 N-channel 30V 5A, Q13 BC817, Q14 BC817, Q2 N-channel 30V 5A, Q3 N-channel 30V 5A, Q4 N-channel 30V 5A, Q5 N-channel 30V 5A, Q6 N-channel 30V 5A, Q7 N-channel 30V 5A, Q8 N-channel 30V 5A, Q9 N-channel 30V 5A, SW1 SW_Push, SW2 SW_Push, U1 DS18B20, U2 ds2438az+, U3 LP38690DT-3.3, U4 SX1308, U5 ESP32-WROOM-32D

Commit message: battery stabilizer capacitor, named switches
Parts:
- added C24: 1000uF, Capacitor_THT:CP_Radial_D10.0mm_P5.00mm, F.Cu at (186.3, 71.2)
- Boot1: renamed from SW2; value SW_Push -> Boot
- moved R16 6.04 mm to (183.5, 78.5), turned to 90 degrees
- moved Q6 2.33 mm to (179.6, 78.5), turned to 180 degrees
- renumbered SW1 to Reset1
Routing:
- net VCC_BATT: track 33.7 -> 96.5 mm
- net Rsense+: track 118.7 -> 135.7 mm
- net GND: track 1291.3 -> 1297.2 mm
- net Net-(Q6-Pad1): track 14.7 -> 9.49 mm
- net Net-(CUSTOM1-Pad3): track 10.2 -> 7.50 mm
- net 3_3V: track 257.5 -> 255.2 mm
- net Temp: track 191.3 -> 192.4 mm
Other:
- board text added: "PlantCtrl V0.8"
- board text removed: "PlantCtrl V0.7"

Commit message: added power supervisor
Parts:
- added R57: 1k, Resistor_SMD:R_0805_2012Metric_Pad1.15x1.40mm_HandSolder, F.Cu at (252.0, 87.8)
- added R60: 19k-19.5K, Resistor_SMD:R_0805_2012Metric_Pad1.15x1.40mm_HandSolder, F.Cu at (255.9, 87.8)
- added U6: CN61CN33, Package_TO_SOT_SMD:SOT-23, F.Cu at (248.2, 86.5)
Connections:
- Q11 pad 1: Net-(IC1-Pad1) -> Net-(Q11-Pad1)
Routing:
- net GND: track 1297.2 -> 1325.6 mm, vias 114 -> 115
- net VCC_BAT_FUSED: track 18.1 -> 30.1 mm
- net Net-(Q11-Pad1): track 0.00 -> 4.56 mm
- net Net-(R57-Pad2): track 0.00 -> 4.24 mm
- net Net-(IC1-Pad1): track 3.82 -> 2.93 mm

Commit message: use correct footprints for oven soldering
Parts:
- C1, C10, C11, C12, C13, C14, C15, C16, C17, C18, C19, C2, C20, C21, C3, C4, C5, C6, C7, C8, C9: footprint Capacitor_SMD:C_0805_2012Metric_Pad1.15x1.40mm_HandSolder -> Capacitor_SMD:C_0805_2012Metric
- D1, D2, D3, D4, D5, D6, D7, Pumps1, Sensor1: footprint LED_SMD:LED_0805_2012Metric_Pad1.15x1.40mm_HandSolder -> LED_SMD:LED_0805_2012Metric_Castellated
- Q1, Q10, Q11, Q12, Q2, Q3, Q4, Q5, Q6, Q7, Q8, Q9, Q_PWR1, Q_PWR2, Q_PWR3: footprint Package_TO_SOT_SMD:SOT-23_Handsoldering -> Package_TO_SOT_SMD:SOT-23
- R1, R10, R11, R12, R13, R14, R15, R16, R17, R18, R19, R2, R20, R21, R22, R23, R24, R25, R26, R27, R28, R29, R3, R30, R31, R32, R33, R34, R35, R36, R37, R38, R39, R4, R40, R41, R42, R43, R44, R45, R46, R47, R48, R49, R5, R50, R51, R52, R53, R54, R55, R56, R57, R58, R59, R6, R60, R7, R8, R9: footprint Resistor_SMD:R_0805_2012Metric_Pad1.15x1.40mm_HandSolder -> Resistor_SMD:R_0805_2012Metric
Routing:
- net PLANT0_MOIST: track 59.1 -> 61.3 mm
- net GND: track 1325.6 -> 1327.5 mm, vias 115 -> 119
- net PLANT5_MOIST: track 100.0 -> 99.0 mm
- net PLANT1_MOIST: track 66.0 -> 65.3 mm
- net PLANT3_MOIST: track 78.0 -> 77.3 mm
- net Net-(Q_PWR1-Pad1): track 4.75 -> 5.34 mm
- net Net-(Q11-Pad1): track 4.56 -> 3.98 mm
- net PLANT6_MOIST: track 110.0 -> 109.4 mm
- net Net-(Q3-Pad1): track 4.39 -> 4.94 mm
- net Net-(Q4-Pad1): track 4.39 -> 4.89 mm
- net LIPO_OC: track 42.3 -> 42.8 mm
- net Net-(Q_PWR3-Pad1): track 4.47 -> 4.97 mm
- net Net-(Q6-Pad1): track 9.49 -> 9.99 mm
- net Net-(Q5-Pad1): track 4.39 -> 4.89 mm
- net Net-(Q2-Pad1): track 4.38 -> 4.88 mm
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
Commit message: 0.9 final
Parts:
- removed Debug1: Conn_01x01_Male, TestPoint:TestPoint_Pad_1.5x1.5mm
- removed GPIO1: Conn_01x04_Female, Connector_JST:JST_EH_B4B-EH-A_1x04_P2.50mm_Vertical
- removed IC1: DW01, misc_footprints:SOT95P280X135-6N
- removed JP2, OCP1: SolderJumper_2_Open, Jumper:SolderJumper-2_P1.3mm_Open_Pad1.0x1.5mm
- removed Q12: N-channel 30V 5A, Package_TO_SOT_SMD:SOT-23
- removed R57: 1k, Resistor_SMD:R_0805_2012Metric
- removed R58: 10k, Resistor_SMD:R_0805_2012Metric
- removed R60: 19k-19.5K, Resistor_SMD:R_0805_2012Metric
- added C25: 1000uF, Capacitor_THT:CP_Radial_D10.0mm_P5.00mm, F.Cu at (199.5, 95.6)
- added D27: BAS40-04, Package_TO_SOT_SMD:SOT-23, F.Cu at (178.8, 82.2)
- R24, R25, R55: value 10k -> 1k
- R31: value 270 -> 4,7K
- R53: value 100 -> 100k
- SOLAR_PWR1: footprint Jumper:SolderJumper-2_P1.3mm_Bridged_Pad1.0x1.5mm -> Jumper:SolderJumper-2_P1.3mm_Open_Pad1.0x1.5mm
- Shunt1: value 0.100 -> 0.025
- moved R25 72.7 mm to (201.4, 79.1)
- moved R24 72.6 mm to (267.8, 108.5)
- moved R55 58.1 mm to (252.9, 82.4), turned to 270 degrees
- moved R52 21.4 mm to (242.3, 78.1), turned to 90 degrees
- moved C10 11.7 mm to (248.2, 82.4), turned to 90 degrees
- moved Q11 9.21 mm to (245.4, 82.4), turned to 0 degrees
- moved U6 8.96 mm to (245.4, 78.0), turned to 0 degrees
- moved R53 8.84 mm to (248.3, 78.0)
- moved I2C1 7.57 mm to (205.9, 104.3), turned to 180 degrees
- moved R16 7.30 mm to (185.2, 85.6), turned to 0 degrees
- moved Q6 5.58 mm to (183.3, 82.7)
- moved D16 4.90 mm to (179.1, 86.5), turned to 0 degrees
- moved R46 3.89 mm to (185.2, 87.6), turned to 0 degrees
Connections:
- net VCC_BAT_FUSED renamed VCC_FUSED_ALWAYS
- CUSTOM1 pad 2: Net-(CUSTOM1-Pad2) -> CUSTOM_GPIO1
- D16 pad 3: CUSTOM_GPIO -> CUSTOM_GPIO1
- Hall1 pad 3: Net-(Debug1-Pad1) -> HALL_RX
- Q11 pad 1: Net-(Q11-Pad1) -> Net-(C10-Pad2)
- Q11 pad 3: enable_all -> Net-(Q11-Pad3)
- R24 pad 1: Net-(Q_PWR1-Pad1) -> Net-(Q_PWR2-Pad1)
- R24 pad 2: Net-(Q9-Pad3) -> Net-(Q10-Pad3)
- R25 pad 1: Net-(Q_PWR2-Pad1) -> Net-(Q_PWR1-Pad1)
- R25 pad 2: Net-(Q10-Pad3) -> Net-(Q9-Pad3)
- R46 pad 2: CUSTOM_GPIO -> GPIO2
- R52 pad 1: SOLAR_GND -> Net-(C10-Pad2)
- R52 pad 2: Net-(IC1-Pad2) -> Net-(R52-Pad2)
- R55 pad 1: Net-(GPIO1-Pad2) -> Net-(Q_PWR3-Pad1)
- R55 pad 2: GND -> Net-(Q11-Pad3)
- SOLAR1 pad 2: SOLAR_GND -> GND
- SOLAR1 pad 3: SOLAR_GND -> GND
- U5 pad 13: Net-(GPIO1-Pad3) -> SENSORS_ENABLE
- U5 pad 23: HALL_TX -> PLANT_CTRL_PUMP_0
- U5 pad 24: Net-(GPIO1-Pad2) -> GPIO2
- U5 pad 26: CUSTOM_GPIO -> CUSTOM_GPIO1
- U5 pad 27: SENSORS_ENABLE -> HALL_TX
- U5 pad 28: PLANT_CTRL_PUMP_0 -> HALL_RX
- U5 pad 6: Net-(I2C1-Pad2) -> Net-(I2C1-Pad3)
- U5 pad 7: Net-(I2C1-Pad3) -> Net-(I2C1-Pad2)
- U6 pad 1: Net-(R57-Pad2) -> Net-(R52-Pad2)
Routing:
- net GND: track 1327.5 -> 1266.8 mm, vias 119 -> 118
- net SOLAR_GND: track 50.9 -> 0.00 mm, vias 1 -> 0
- net HALL_RX: track 0.00 -> 46.5 mm, vias 0 -> 2
- net Net-(GPIO1-Pad3): track 46.2 -> 0.00 mm, vias 1 -> 0
- net LIPO_OC: track 42.8 -> 0.00 mm
- net PWR_SENSORS: track 194.3 -> 160.9 mm
- net GPIO2: track 0.00 -> 22.3 mm, vias 0 -> 2
- net CUSTOM_GPIO1: track 0.00 -> 20.9 mm, vias 0 -> 2
- net Net-(GPIO1-Pad2): track 20.5 -> 0.00 mm
- net CUSTOM_GPIO: track 19.1 -> 0.00 mm, vias 2 -> 0
- net Net-(Q11-Pad3): track 0.00 -> 14.7 mm
- net SENSORS_ENABLE: track 81.1 -> 67.0 mm
- net 3_3V: track 254.8 -> 267.0 mm, vias 8 -> 7
- net VCC: track 264.9 -> 275.7 mm, vias 8 -> 7
- net HALL_TX: track 35.3 -> 45.1 mm
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Other:
- board text added: "PlantCtrl V0.9"
- board text removed: "PlantCtrl V0.8"

Commit message: more capacitors, slight layout optimisation
Parts:
- added C26: 1000uF, Capacitor_THT:CP_Radial_D10.0mm_P5.00mm, F.Cu at (213.1, 86.4)
- added D28: BAS40-04, Package_TO_SOT_SMD:SOT-23, F.Cu at (174.0, 62.2)
- R26: value 4k7 -> 2.2k
- moved Pumps1 2.59 mm to (210.3, 114.0)
Connections:
- J1 pad 4: (no net) -> Net-(J1-Pad4)
- U2 pad 6: (no net) -> Net-(U2-Pad6)
- U2 pad 7: (no net) -> Net-(U2-Pad7)
- U4 pad 6: (no net) -> Net-(U4-Pad6)
- U5 pad 14: Temp -> CUSTOM_GPIO1
- U5 pad 17: (no net) -> Net-(U5-Pad17)
- U5 pad 18: (no net) -> Net-(U5-Pad18)
- U5 pad 19: (no net) -> Net-(U5-Pad19)
- U5 pad 20: (no net) -> Net-(U5-Pad20)
- U5 pad 21: (no net) -> Net-(U5-Pad21)
- U5 pad 22: (no net) -> Net-(U5-Pad22)
- U5 pad 26: CUSTOM_GPIO1 -> Temp
- U5 pad 32: (no net) -> Net-(U5-Pad32)
Routing:
- net 3_3V: track 267.0 -> 272.4 mm, vias 7 -> 9
- net Temp: track 191.4 -> 196.2 mm
- net VCC: track 275.7 -> 280.3 mm
- net Net-(Pumps1-Pad2): track 2.08 -> 5.36 mm
- net GND: track 1266.8 -> 1269.8 mm

Commit message: changed switches to cheaper alternative
Parts:
- Boot1, Reset1: footprint Button_Switch_SMD:SW_Push_1P1T_NO_CK_KMR2 -> Button_Switch_SMD:SW_SPST_CK_RS282G05A3
- moved C18 4.08 mm to (177.8, 137.4)
- moved Boot1 1.97 mm to (196.0, 137.5)
- moved Reset1 1.95 mm to (184.0, 137.5)
Connections:
- J1 pad 4: Net-(J1-Pad4) -> (no net)
- U2 pad 6: Net-(U2-Pad6) -> (no net)
- U2 pad 7: Net-(U2-Pad7) -> (no net)
- U4 pad 6: Net-(U4-Pad6) -> (no net)
- U5 pad 17: Net-(U5-Pad17) -> (no net)
- U5 pad 18: Net-(U5-Pad18) -> (no net)
- U5 pad 19: Net-(U5-Pad19) -> (no net)
- U5 pad 20: Net-(U5-Pad20) -> (no net)
- U5 pad 21: Net-(U5-Pad21) -> (no net)
- U5 pad 22: Net-(U5-Pad22) -> (no net)
- U5 pad 32: Net-(U5-Pad32) -> (no net)
Routing:
- net 3_3V: track 272.4 -> 267.8 mm
- net GND: track 1269.8 -> 1266.1 mm, vias 118 -> 116
- net Net-(C2-Pad2): track 79.3 -> 82.6 mm
- net Net-(C18-Pad2): track 8.47 -> 7.77 mm

Commit message: fixed power on download mode, solar voltage sensor fixed
Parts:
- removed EN1, IO0_1: NC, Jumper:SolderJumper-2_P1.3mm_Bridged_Pad1.0x1.5mm
- removed Q13, Q14: BC817, Package_TO_SOT_SMD:SOT-23
- removed R20, R56: 10k, Resistor_SMD:R_0805_2012Metric
- J1: value Conn_01x06_Female -> Conn_01x03_Female; footprint Connector_PinHeader_2.54mm:PinHeader_1x06_P2.54mm_Vertical -> Connector_PinHeader_2.54mm:PinHeader_1x03_P2.54mm_Vertical
- R2, R48: value 10k -> 1k
- R54: value 100k -> 10k
- moved R54 81.6 mm to (182.1, 86.6), turned to 90 degrees
- moved J1 12.7 mm to (207.0, 109.7), turned to 270 degrees
Connections:
- J1 pad 1: DTR -> GND
- R4 pad 1: Net-(R4-Pad1) -> Net-(C21-Pad1)
- R48 pad 2: Net-(R4-Pad1) -> Net-(C21-Pad1)
- R54 pad 1: Net-(R4-Pad1) -> CUSTOM_GPIO1
- R54 pad 2: Net-(C21-Pad1) -> GND
- U2 pad 6: (no net) -> Net-(U2-Pad6)
- U2 pad 7: (no net) -> Net-(U2-Pad7)
- U4 pad 6: (no net) -> Net-(U4-Pad6)
- U5 pad 17: (no net) -> Net-(U5-Pad17)
- U5 pad 18: (no net) -> Net-(U5-Pad18)
- U5 pad 19: (no net) -> Net-(U5-Pad19)
- U5 pad 20: (no net) -> Net-(U5-Pad20)
- U5 pad 21: (no net) -> Net-(U5-Pad21)
- U5 pad 22: (no net) -> Net-(U5-Pad22)
- U5 pad 32: (no net) -> Net-(U5-Pad32)
Routing:
- net CUSTOM_GPIO1: track 20.9 -> 46.5 mm, vias 2 -> 1
- net Net-(C19-Pad2): track 48.6 -> 25.1 mm, vias 2 -> 0
- net Net-(C21-Pad1): track 4.43 -> 26.4 mm
- net IO0: track 20.1 -> 0.00 mm, vias 2 -> 0
- net Temp: track 196.2 -> 176.9 mm
- net Net-(R4-Pad1): track 18.1 -> 0.00 mm
- net EN: track 17.9 -> 0.00 mm, vias 2 -> 0
- net Net-(C2-Pad2): track 82.6 -> 68.5 mm, vias 3 -> 2
- net Net-(Q13-Pad2): track 11.5 -> 0.00 mm
- net GND: track 1266.1 -> 1275.9 mm
- net DTR: track 8.64 -> 0.00 mm
- net ESP_TX: track 33.2 -> 41.8 mm
- net RTS: track 5.78 -> 0.00 mm
- net Net-(Q14-Pad2): track 5.32 -> 0.00 mm
- net ESP_RX: track 33.8 -> 36.4 mm
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