File: board/PlantCtrlESP32.kicad_pcb (KiCad board)
At the start: 2 copper layers, 99.1 x 99.1 mm, 163 parts, among them J1 Conn_01x03_Female, Q1 N-channel 30V 5A, Q10 N-channel 30V 5A, Q11 N-channel 30V 5A, Q2 N-channel 30V 5A, Q3 N-channel 30V 5A, Q4 N-channel 30V 5A, Q5 N-channel 30V 5A, Q6 N-channel 30V 5A, Q7 N-channel 30V 5A, Q8 N-channel 30V 5A, Q9 N-channel 30V 5A, U1 DS18B20, U2 ds2438az+, U3 LP38690DT-3.3, U4 SX1308, U5 ESP32-WROOM-32D, U6 CN61CN33

Commit message: add high impendance pulldown to analog in
Parts:
- added R20: 100k, Resistor_SMD:R_0805_2012Metric, F.Cu at (218.7, 130.3)
- added R56: 100k, Resistor_SMD:R_0805_2012Metric, F.Cu at (226.4, 130.3)
- added R57: 100k, Resistor_SMD:R_0805_2012Metric, F.Cu at (234.1, 130.3)
- added R58: 100k, Resistor_SMD:R_0805_2012Metric, F.Cu at (241.6, 130.3)
- added R60: 100k, Resistor_SMD:R_0805_2012Metric, F.Cu at (249.2, 130.4)
- added R61: 100k, Resistor_SMD:R_0805_2012Metric, F.Cu at (256.8, 130.4)
- added R62: 100k, Resistor_SMD:R_0805_2012Metric, F.Cu at (264.3, 130.3)
Routing:
- net GND: track 1322.8 -> 1354.6 mm
- net Net-(R45-Pad1): track 5.67 -> 7.86 mm
- net Net-(R43-Pad1): track 5.67 -> 7.86 mm
- net Net-(R49-Pad1): track 5.56 -> 7.75 mm
- net Net-(R37-Pad1): track 5.77 -> 7.84 mm
- net Net-(R20-Pad2): track 5.88 -> 7.96 mm
- net Net-(R41-Pad1): track 5.67 -> 7.73 mm
- net Net-(R39-Pad1): track 5.79 -> 7.86 mm

Commit message: reduced odd resistors
Parts:
- added R63: 1k, Resistor_SMD:R_0805_2012Metric, F.Cu at (181.2, 77.7)
- added R64: 10k, Resistor_SMD:R_0805_2012Metric, F.Cu at (206.6, 126.1)
- R26: value 2.2k -> 1k
- R31: value 4,7K -> 10k
- moved R31 7.12 mm to (203.3, 126.1), turned to 90 degrees
- moved R26 3.64 mm to (178.2, 77.0), turned to 90 degrees
Connections:
- R26 pad 1: Temp -> Net-(R26-Pad1)
Routing:
- net PWR_SENSORS: track 115.0 -> 125.0 mm
- net Net-(R31-Pad1): track 3.01 -> 8.00 mm
- net GND: track 1354.6 -> 1351.2 mm, vias 117 -> 116
- net Net-(R26-Pad1): track 0.00 -> 2.18 mm
- net 3_3V: track 269.6 -> 271.2 mm
- net Temp: track 176.9 -> 177.4 mm

Commit message: further reduced only once used parts
Parts:
- added R65: 10k, Resistor_SMD:R_0805_2012Metric, F.Cu at (222.8, 72.5)
- R21: value 19k-19.5K -> 10k
- moved R29 1.20 mm to (224.9, 72.5), turned to 270 degrees
- moved R21 0.13 mm to (222.8, 76.2)
Connections:
- R29 pad 1: Net-(R21-Pad2) -> Net-(R29-Pad1)
- U4 pad 3: Net-(R21-Pad2) -> Net-(R29-Pad1)
Routing:
- net Net-(R29-Pad1): track 0.00 -> 5.03 mm
- net Net-(R21-Pad2): track 4.20 -> 1.81 mm
- net PWR_PUMP_CONVERTER: track 138.4 -> 137.6 mm

Commit message: added more correct pull down for download mode
Parts:
- added R66: 1k, Resistor_SMD:R_0805_2012Metric, F.Cu at (198.8, 132.2)
- moved R2 0.16 mm to (195.1, 132.2)
Connections:
- R2 pad 2: 3_3V -> Net-(R2-Pad2)
Routing:
- net GND: track 1351.1 -> 1346.3 mm
- net 3_3V: track 271.2 -> 273.8 mm
- net Net-(R2-Pad2): track 0.00 -> 1.85 mm

Commit message: added distance sensor and adjusted pcb for it
Parts:
- removed Hall1: Conn_01x04, ESP32:SR04M-2PinHeader_1x04_P2.54mm_Vertical
- removed LED_SENS1: NC, Jumper:SolderJumper-2_P1.3mm_Bridged_Pad1.0x1.5mm
- added D29: BAS40-04, Package_TO_SOT_SMD:SOT-23, F.Cu at (204.0, 129.5)
- added I2C1: Conn_01x04, Connector_JST:JST_EH_B4B-EH-A_1x04_P2.50mm_Vertical, F.Cu at (198.6, 128.8)
- added Q12: N-channel 30V 5A, Package_TO_SOT_SMD:SOT-23, F.Cu at (208.0, 137.7)
- added Q_PWR4: P-channel 50v 4A, Package_TO_SOT_SMD:SOT-23, F.Cu at (204.0, 133.1)
- added R67: R, Resistor_SMD:R_0805_2012Metric, F.Cu at (184.4, 125.7)
- added R68: R, Resistor_SMD:R_0805_2012Metric, F.Cu at (186.9, 125.7)
- added R69: 1k, Resistor_SMD:R_0805_2012Metric, F.Cu at (208.0, 132.3)
- added R70: 10k, Resistor_SMD:R_0805_2012Metric, F.Cu at (208.0, 134.6)
- added R71: 1k, Resistor_SMD:R_0805_2012Metric, F.Cu at (204.0, 138.4)
- added R72: 10k, Resistor_SMD:R_0805_2012Metric, F.Cu at (204.0, 136.1)
- moved R31 0.38 mm to (203.3, 125.7)
- moved R64 0.38 mm to (206.6, 125.7)
- renumbered I2C1 to Custom1
Connections:
- Sensor1 pad 1: Net-(LED_SENS1-Pad1) -> GND
- U5 pad 27: HALL_TX -> SCL
- U5 pad 28: HALL_RX -> SDA
Routing:
- net SCL: track 0.00 -> 53.4 mm, vias 0 -> 3
- net SDA: track 0.00 -> 51.5 mm, vias 0 -> 2
- net HALL_RX: track 46.5 -> 0.00 mm, vias 2 -> 0
- net HALL_TX: track 45.1 -> 0.00 mm, vias 2 -> 0
- net PWR_SENSORS: track 125.0 -> 90.8 mm
- net PWR_I2C: track 0.00 -> 27.7 mm
- net SENSORS_ENABLE: track 67.0 -> 81.0 mm, vias 0 -> 2
- net 3_3V: track 273.8 -> 286.8 mm
- net GND: track 1346.3 -> 1357.5 mm, vias 116 -> 114
- net Net-(Q_PWR4-Pad1): track 0.00 -> 4.35 mm
- net Net-(Q12-Pad1): track 0.00 -> 4.35 mm
- net Net-(Q12-Pad3): track 0.00 -> 3.25 mm
- net Net-(LED_SENS1-Pad1): track 2.66 -> 0.00 mm
- net VCC: track 280.3 -> 282.6 mm

Commit message: new extension header, improved labeling of connectors, optimized layout
Parts:
- removed CUSTOM1: Conn_01x04, Connector_JST:JST_EH_B4B-EH-A_1x04_P2.50mm_Vertical
- removed Custom1: Conn_01x04_Female, Connector_JST:JST_EH_B4B-EH-A_1x04_P2.50mm_Vertical
- added 12V1: SolderJumper_2_Open, Jumper:SolderJumper-2_P1.3mm_Open_Pad1.0x1.5mm, F.Cu at (207.6, 109.2)
- added 12V2: SolderJumper_2_Open, Jumper:SolderJumper-2_P1.3mm_Open_Pad1.0x1.5mm, F.Cu at (205.1, 85.7)
- added 3_3V1: SolderJumper_2_Open, Jumper:SolderJumper-2_P1.3mm_Open_Pad1.0x1.5mm, F.Cu at (202.6, 109.2)
- added 3_3V2: SolderJumper_2_Open, Jumper:SolderJumper-2_P1.3mm_Open_Pad1.0x1.5mm, F.Cu at (200.0, 85.7)
- added D30: BAS40-04, Package_TO_SOT_SMD:SOT-23, F.Cu at (205.0, 103.9)
- added D31: BAS40-04, Package_TO_SOT_SMD:SOT-23, F.Cu at (198.1, 111.1)
- added D32: BAS40-04, Package_TO_SOT_SMD:SOT-23, F.Cu at (202.6, 81.9)
- added J2: Conn_02x04_Counter_Clockwise, Connector_PinHeader_2.54mm:PinHeader_2x04_P2.54mm_Vertical, F.Cu at (198.8, 98.4)
- added Q13: N-channel 30V 5A, Package_TO_SOT_SMD:SOT-23, F.Cu at (189.8, 85.7)
- added Q_PWR5: P-channel 50v 4A, Package_TO_SOT_SMD:SOT-23, F.Cu at (200.7, 103.9)
- added Q_PWR6: P-channel 50v 4A, Package_TO_SOT_SMD:SOT-23, F.Cu at (196.2, 83.2)
- added R73: 10k, Resistor_SMD:R_0805_2012Metric, F.Cu at (197.6, 103.9)
- added R74: 1k, Resistor_SMD:R_0805_2012Metric, F.Cu at (186.8, 85.7)
- added R75: 10k, Resistor_SMD:R_0805_2012Metric, F.Cu at (187.6, 82.5)
- added R76: 1k, Resistor_SMD:R_0805_2012Metric, F.Cu at (193.7, 86.4)
- added R77: 10k, Resistor_SMD:R_0805_2012Metric, F.Cu at (193.0, 83.2)
- added VCC1: SolderJumper_2_Open, Jumper:SolderJumper-2_P1.3mm_Open_Pad1.0x1.5mm, F.Cu at (205.1, 109.2)
- added VCC2: SolderJumper_2_Open, Jumper:SolderJumper-2_P1.3mm_Open_Pad1.0x1.5mm, F.Cu at (202.6, 85.7)
- R16, R54: value 10k -> 1k
- R46: value 1k -> 10k
- SOLAR_PWR1: value NC -> NO
- moved D16 43.6 mm to (185.9, 129.5), turned to 180 degrees
- moved D27 32.8 mm to (194.3, 111.1), turned to 90 degrees
- moved C25 24.8 mm to (176.5, 86.4)
- moved R54 20.3 mm to (194.3, 102.9), turned to 180 degrees
- moved Q6 18.3 mm to (194.3, 97.3), turned to 270 degrees
- moved D28 17.8 mm to (173.4, 80.0), turned to 0 degrees
- moved R16 17.6 mm to (194.3, 100.6), turned to 180 degrees
- moved Pumps1 11.6 mm to (208.3, 102.6)
- moved R46 11.3 mm to (194.3, 94.2), turned to 180 degrees
- moved J1 5.98 mm to (205.7, 115.6)
- moved C23 5.69 mm to (224.8, 86.4), turned to 0 degrees
- moved R30 4.06 mm to (210.8, 102.9)
- moved C2 2.24 mm to (189.6, 92.6), turned to 0 degrees
- moved R25 0.40 mm to (201.3, 78.7), turned to 180 degrees
Connections:
- D16 pad 2: 3_3V -> VCC
- D16 pad 3: CUSTOM_GPIO1 -> 3_3V
- D27 pad 2: VCC -> 3_3V
- D27 pad 3: Net-(CUSTOM1-Pad3) -> CUSTOM_GPIO34
- Q6 pad 3: Net-(CUSTOM1-Pad3) -> Net-(Q6-Pad3)
- R16 pad 2: GND -> CUSTOM_GPIO2
- R46 pad 2: GPIO2 -> GND
- R54 pad 1: CUSTOM_GPIO1 -> Net-(Q_PWR5-Pad1)
- R54 pad 2: GND -> Net-(Q6-Pad3)
- U2 pad 6: (no net) -> Net-(U2-Pad6)
- U2 pad 7: (no net) -> Net-(U2-Pad7)
- U4 pad 6: (no net) -> Net-(U4-Pad6)
- U5 pad 14: CUSTOM_GPIO1 -> CUSTOM_GPIO12
- U5 pad 17: (no net) -> Net-(U5-Pad17)
- U5 pad 18: (no net) -> Net-(U5-Pad18)
- U5 pad 19: (no net) -> Net-(U5-Pad19)
- U5 pad 20: (no net) -> Net-(U5-Pad20)
- U5 pad 21: (no net) -> Net-(U5-Pad21)
- U5 pad 22: (no net) -> Net-(U5-Pad22)
- U5 pad 24: GPIO2 -> CUSTOM_GPIO2
- U5 pad 32: (no net) -> Net-(U5-Pad32)
- U5 pad 6: Net-(Custom1-Pad3) -> CUSTOM_GPIO34
- U5 pad 7: Net-(Custom1-Pad2) -> CUSTOM_GPIO35
Routing:
- net CUSTOM_GPIO1: track 46.5 -> 0.00 mm, vias 1 -> 0
- net PUMP_PWR: track 201.4 -> 240.4 mm, vias 2 -> 5
- net CUSTOM_GPIO35: track 0.00 -> 38.2 mm, vias 0 -> 2
- net CUSTOM_GPIO34: track 0.00 -> 36.6 mm, vias 0 -> 2
- net Net-(D32-Pad3): track 0.00 -> 35.1 mm, vias 0 -> 1
- net Net-(Custom1-Pad2): track 32.5 -> 0.00 mm, vias 1 -> 0
- net CUSTOM_GPIO12: track 0.00 -> 32.4 mm, vias 0 -> 2
- net Net-(Custom1-Pad3): track 30.0 -> 0.00 mm, vias 1 -> 0
- net 3_3V: track 286.8 -> 314.8 mm
- net GND: track 1357.5 -> 1381.4 mm, vias 114 -> 127
- net GPIO2: track 22.3 -> 0.00 mm, vias 2 -> 0
- net Net-(12V1-Pad1): track 0.00 -> 19.8 mm
- net VCC: track 282.6 -> 265.3 mm
- net Net-(12V2-Pad1): track 0.00 -> 15.4 mm
- net Net-(D30-Pad3): track 0.00 -> 10.1 mm
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Other:
- board text added: "12V GND"
- board text added: "34 35 2 12"
- board text added: "3V3 D GND"
- board text added: "GND 3V3 VCC 12V"
- board text added: "GND VCC S"
- board text added: "GPIO12"
- board text added: "GPIO2"
- board text added: "IN GND GND VCC"
- board text added: "RX TX GND"

Commit message: 0.10 rev final
Parts:
- renumbered C23 to C10, C22 to C11, C11 to C12, C24 to C13, C10 to C14, C26 to C15, C20 to C16, C21 to C17, C14 to C18, C16 to C19, C17 to C2, C3 to C20, C4 to C21, C5 to C22, C6 to C23, C7 to C24, C8 to C25, C9 to C26, C15 to C3, C2 to C4, C18 to C5, C19 to C6, C13 to C7, C25 to C8, C12 to C9, D27 to D1, D1 to D10, D2 to D11, D4 to D12, D6 to D13, D3 to D14, D5 to D15, D7 to D16, D14 to D17, D17 to D18, D20 to D19, D31 to D2, D21 to D20, D22 to D21, D23 to D22, D24 to D23, D29 to D24, D9 to D26, D10 to D27, D11 to D28, D12 to D29, D28 to D3, D13 to D30, D15 to D31, D19 to D32, D30 to D4, D32 to D5, D16 to D6, D8 to D7, D26 to D8, D18 to D9, J2 to J1, J1 to J2, LIPO2 to LIPO1, LIPO1 to LIPO2, PUMP0 to PUMP1, PUMP1 to PUMP2, PUMP2 to PUMP3, PUMP3 to PUMP4, PUMP4 to PUMP5, PUMP5 to PUMP6, PUMP6 to PUMP7, Q6 to Q1, Q5 to Q10, Q8 to Q11, Q10 to Q13, Q13 to Q2, Q9 to Q3, Q11 to Q4, Q1 to Q5, Q2 to Q6, Q4 to Q7, Q7 to Q8, Q3 to Q9, Q_PWR5 to Q_PWR1, Q_PWR6 to Q_PWR2, Q_PWR1 to Q_PWR3, Q_PWR3 to Q_PWR4, Q_PWR4 to Q_PWR5, Q_PWR2 to Q_PWR6, R26 to R1, R75 to R10, R67 to R11, R68 to R12, R1 to R13, R2 to R14, R66 to R15, R33 to R16, R32 to R17, R21 to R18, R65 to R19, R63 to R2, R29 to R20, R30 to R21, R25 to R22, R55 to R23, R53 to R24, R27 to R25, R59 to R26, R50 to R27, R52 to R28, R22 to R29, R54 to R3, R3 to R30, R5 to R31, R7 to R32, R11 to R33, R15 to R34, R9 to R35, R13 to R36, R18 to R37, R4 to R38, R34 to R39, R76 to R4, R36 to R40, R38 to R41, R48 to R42, R40 to R43, R42 to R44, R44 to R45, R47 to R46, R6 to R47, R8 to R48, R12 to R49, R16 to R5, R17 to R50, R10 to R51, R14 to R52, R19 to R53, R20 to R54, R35 to R55, R37 to R57, R57 to R58, R39 to R59, R74 to R6, R58 to R60, R41 to R61, R60 to R62, R43 to R63, R61 to R64, R45 to R65, R62 to R66, R49 to R67, R31 to R68, R64 to R69, R73 to R7, R71 to R70, R24 to R71, R28 to R73, R69 to R74, R51 to R75, R70 to R76, R23 to R77, R77 to R8, R46 to R9, S0 to S1, S1 to S2, S2 to S3, S3 to S4, S4 to S5, S5 to S6, S6 to S7, U3 to U2, U4 to U3, U5 to U4, U6 to U5, U2 to U6
