File: board/PlantCtrlESP32.kicad_sch (KiCad schematic)
At the start: 405 parts, among them J2 Conn_01x02_Male, J2 Conn_01x03_Female, J2 Conn_01x07, Q12 N-channel 30V 5A, Q2 N-channel 30V 5A, Q3 N-channel 30V 5A, U1 74HC595, U1 AP63200, U1 AP63203, U1 TLC555xP, U2 74HC595, U34 HT7550-1-SOT89, U35 LM393, U36 PC817, U4 ESP32-WROOM-32D

Commit message: layouting continued
Parts:
- added TP8: LED-Enabled, TestPoint:TestPoint_THTPad_D2.0mm_Drill1.0mm, symbol Connector:TestPoint
- C72: footprint (none) -> Capacitor_SMD:C_0603_1608Metric
- J2: footprint (none) -> Connector_PinHeader_2.54mm:PinHeader_1x07_P2.54mm_Horizontal
- R23, R24: footprint (none) -> Resistor_SMD:R_0603_1608Metric
- Test_Solar_In1: footprint (none) -> Button_Switch_SMD:SW_SPST_CK_RS282G05A3
Connections:
- net SIGNAL_NEXT is gone; now on net SIGNAL: D23.3, J2.4 (Pin_4), TP25.1
- net LED_ENABLE: now also U4.11 (IO26), TP8.1
Changed lines of the file:
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@@
   (junction (at 174.625 602.615) (diameter 0) (color 0 0 0 0)
   )
+  (junction (at 44.704 594.995) (diameter 0) (color 0 0 0 0)
+  )
   (junction (at 319.278 156.718) (diameter 0) (color 0 0 0 0)
   )
@@
     (stroke (width 0) (type default))
   )
+  (wire (pts (xy 44.704 594.995) (xy 45.085 594.995))
+    (stroke (width 0) (type default))
+  )
   (wire (pts (xy 353.568 210.058) (xy 368.808 210.058))
     (stroke (width 0) (type default))
@@
     (stroke (width 0) (type default))
   )
-  (wire (pts (xy 43.815 594.995) (xy 45.085 594.995))
+  (wire (pts (xy 43.815 594.995) (xy 44.704 594.995))
     (stroke (width 0) (type default))
   )
@@
     )
   )
-  (global_label "SIGNAL_NEXT" (shape input) (at 485.648 303.784 180) (fields_autoplaced)
+  (global_label "SIGNAL" (shape input) (at 485.648 303.784 180) (fields_autoplaced)
     (effects (font (size 1.27 1.27)) (justify right))
-    (property "Intersheetrefs" "${INTERSHEET_REFS}" (at 471.2407 303.784 0)
+    (property "Intersheetrefs" "${INTERSHEET_REFS}" (at 476.8649 303.784 0)
       (effects (font (size 1.27 1.27)) (justify right) hide)
     )
@@
     )
   )
+  (global_label "LED_ENABLE" (shape input) (at 107.696 120.142 0) (fields_autoplaced)
+    (effects (font (size 1.27 1.27)) (justify left))
+    (property "Intersheetrefs" "${INTERSHEET_REFS}" (at 121.3775 120.142 0)
+      (effects (font (size 1.27 1.27)) (justify left) hide)
+    )
+  )
   (global_label "GND" (shape input) (at 744.728 149.098 0) (fields_autoplaced)
     (effects (font (size 1.27 1.27)) (justify left))
@@
       (effects (font (size 1.27 1.27)) (justify left))
     )
-    (property "Footprint" "" (at 156.337 591.185 90)
+    (property "Footprint" "Resistor_SMD:R_0603_1608Metric" (at 156.337 591.185 90)
       (effects (font (size 1.27 1.27)) hide)
     )
@@
       (effects (font (size 1.27 1.27)) (justify left))
     )
-    (property "Footprint" "" (at 528.828 303.784 0)
+    (property "Footprint" "Connector_PinHeader_2.54mm:PinHeader_1x07_P2.54mm_Horizontal" (at 528.828 303.784 0)
       (effects (font (size 1.27 1.27)) hide)
     )
@@
     )
   )
+  (symbol (lib_id "Connector:TestPoint") (at 44.704 594.995 0) (unit 1)
+    (in_bom yes) (on_board yes) (dnp no) (fields_autoplaced)
+    (property "Reference" "TP8" (at 46.228 591.058 0)
+      (effects (font (size 1.27 1.27)) (justify left))
+    )
+    (property "Value" "LED-Enabled" (at 46.228 593.598 0)
+      (effects (font (size 1.27 1.27)) (justify left))
+    )
+    (property "Footprint" "TestPoint:TestPoint_THTPad_D2.0mm_Drill1.0mm" (at 49.784 594.995 0)
+      (effects (font (size 1.27 1.27)) hide)
+    )
+    (property "Datasheet" "~" (at 49.784 594.995 0)
+      (effects (font (size 1.27 1.27)) hide)
+    )
+    (pin "1")
+    (instances
+      (project "PlantCtrlESP32"
+        (path "/c26e8d55-0b6e-4c4e-b7c8-b1fed973201c"
+          (reference "TP8") (unit 1)
+        )
+      )
+    )
+  )
   (symbol (lib_id "Connector_Generic:Conn_01x02") (at 388.112 372.618 90) (unit 1)
     (in_bom yes) (on_board yes) (dnp no) (fields_autoplaced)
@@
       (effects (font (size 1.27 1.27)) (justify left))
     )
-    (property "Footprint" "" (at 156.337 582.295 90)
+    (property "Footprint" "Resistor_SMD:R_0603_1608Metric" (at 156.337 582.295 90)
       (effects (font (size 1.27 1.27)) hide)
     )
@@
       (effects (font (size 1.27 1.27)) (justify right))
     )
-    (property "Footprint" "" (at 202.692 744.22 0)
+    (property "Footprint" "Button_Switch_SMD:SW_SPST_CK_RS282G05A3" (at 202.692 744.22 0)
       (effects (font (size 1.27 1.27)) hide)
     )
@@
       (effects (font (size 1.27 1.27)) (justify left))
     )
-    (property "Footprint" "" (at 150.1902 586.105 0)
+    (property "Footprint" "Capacitor_SMD:C_0603_1608Metric" (at 150.1902 586.105 0)
       (effects (font (size 1.27 1.27)) hide)
     )
