File: board/PlantCtrlESP32.kicad_sch (KiCad schematic)
At the start: 406 parts, among them J2 Conn_01x02_Male, J2 Conn_01x03_Female, J2 Conn_01x07, Q12 N-channel 30V 5A, Q2 N-channel 30V 5A, Q3 N-channel 30V 5A, U1 74HC595, U1 AP63200, U1 AP63203, U1 TLC555xP, U2 74HC595, U34 HT7550-1-SOT89, U35 LM393, U36 PC817, U4 ESP32-WROOM-32D

Commit message: add charging circuit
Parts:
- removed C9: 22uf, symbol Device:C
- removed CentralPump/Valve1, Solar_In1: Conn_01x02, symbol Connector_Generic:Conn_01x02
- removed D1, D75: D, symbol Device:D
- removed D13, D74: GREEN, LED_SMD:LED_0603_1608Metric, symbol Device:LED
- removed D4: RED, LED_SMD:LED_0603_1608Metric, symbol Device:LED
- removed D76: YELLOW, LED_SMD:LED_0603_1608Metric, symbol Device:LED
- removed F2: Fuse, symbol Device:Fuse
- removed Half_Solar_IN1: TestPoint, symbol Connector:TestPoint
- removed R29, R75, R77: 1k, Resistor_SMD:R_0603_1608Metric, symbol Device:R
- removed R31, R73: 10k, Resistor_SMD:R_0603_1608Metric, symbol Device:R
- removed TP1: Solar_IN, TestPoint:TestPoint_THTPad_D2.0mm_Drill1.0mm, symbol Connector:TestPoint
- removed TP2: Solar_GND, TestPoint:TestPoint_THTPad_D2.0mm_Drill1.0mm, symbol Connector:TestPoint
- removed TP3: Solar_3V3 LDO, TestPoint:TestPoint_THTPad_D2.0mm_Drill1.0mm, symbol Connector:TestPoint
- removed TP5: IsDay, TestPoint:TestPoint_THTPad_D2.0mm_Drill1.0mm, symbol Connector:TestPoint
- removed Test_Solar_In1: SW_Push, Button_Switch_SMD:SW_SPST_CK_RS282G05A3, symbol Switch:SW_Push
- removed U34: HT7550-1-SOT89, Package_TO_SOT_SMD:SOT-89-3, symbol Regulator_Linear:HT75xx-1-SOT89
- removed U35: LM393, symbol Comparator:LM393
- added BatteryIn1, SolarIn1: TestPoint, symbol Connector:TestPoint
- added C73: 100nF, Capacitor_SMD:C_1206_3216Metric, symbol Device:C
- added C74: 200nF, Capacitor_SMD:C_0603_1608Metric, symbol Device:C
- added C75: C, symbol Device:C
- added C76, C77: C_Polarized, Capacitor_THT:CP_Radial_D13.0mm_P5.00mm, symbol Device:C_Polarized
- added D1: 7v zehner, Diode_SMD:D_SOD-123, symbol Device:D_Zener
- added D100, D101: SS54, Diode_SMD:D_SMB-SMC_Universal_Handsoldering, symbol Device:D_Schottky
- added D98: LED, LED_SMD:LED_0603_1608Metric, symbol Device:LED
- added F1, F3: 4A, symbol Device:Fuse
- added J1: Conn_01x02_Pin, Connector_AMASS:AMASS_XT30UPB-M_1x02_P5.0mm_Vertical, symbol Connector:Conn_01x02_Pin
- added J3: Conn_01x02_Socket, Connector_AMASS:AMASS_XT30UPB-F_1x02_P5.0mm_Vertical, symbol Connector:Conn_01x02_Socket
- added L3: L, Inductor_SMD:L_12x12mm_H4.5mm, symbol Device:L
- added Q6: 4435, Package_SO:SOP-8_3.9x4.9mm_P1.27mm, symbol Simulation_SPICE:PMOS
- added R25: 10k, Resistor_SMD:R_0603_1608Metric, symbol Device:R
- added R27: R_MPPT_LOW, Resistor_SMD:R_0603_1608Metric, symbol Device:R
- added R28: 120, Resistor_SMD:R_0603_1608Metric, symbol Device:R
- added R30, R32: R, Resistor_SMD:R_0603_1608Metric, symbol Device:R
- added R33: 0.06, Resistor_SMD:R_Shunt_Vishay_WSK2512_6332Metric_T1.19mm, symbol Device:R_Shunt
- added R_MPPT_HIGH1: 34k, Resistor_SMD:R_0603_1608Metric, symbol Device:R
- added U6: CN3795, kicad-stuff:SSOP10, symbol CN3795:CN3795
- D11: value 3A 12V -> SS54; footprint (none) -> Diode_SMD:D_SMB-SMC_Universal_Handsoldering
- ExtCharge1: renamed from PowerIn1; footprint (none) -> Connector_AMASS:AMASS_XT30UPB-M_1x02_P5.0mm_Vertical
Connections:
- net 12V: now also F3.1; no longer D11.1 (K)
- net GND: now also ExtCharge1.1 (Pin_1), U36.2, C74.2, C75.2, C76.2, C77.2, D100.2 (A), J1.2 (Pin_2), J3.1 (Pin_1), R27.1, R32.2, U6.2 (GND)
- net S_VIN: now also C73.1, C77.1, D1.1 (K), J1.1 (Pin_1), Q6.3 (S), R25.1, R_MPPT_HIGH1.1, SolarIn1.1, U6.9 (VCC)
- net at D11.2 (A), ExtCharge1.2 (Pin_2): now also D10.2 (A); no longer D10.1 (K)
- net at R9.2: now also D10.1 (K); no longer D10.2 (A)
- net at R8.1: now also D1.2 (A)
- net at R8.2: now also U36.1
- new net: BatteryIn1.1, C75.1, C76.1, D11.1 (K), F1.1, F3.2, R33.1
- new net: R28.1, U6.5 (COM)
- new net: C74.1, R28.2
- new net: C73.2, U6.1 (VG)
- new net: F1.2, J3.2 (Pin_2)
- new net: Q6.2 (G), U6.10 (DRV)
- new net: D98.1 (K), U6.3 (~{CHRG})
- new net: R27.2, R_MPPT_HIGH1.2, U6.4 (MPPT)
- new net: R30.2, R32.1, U6.6 (FB)
- new net: R30.1, R33.2, U6.7 (BAT)
- new net: R33.3, U6.8 (CSP)
- new net: D98.2 (A), R25.2
- new net: D101.2 (A), Q6.1 (D)
- new net: D100.1 (K), D101.1 (K), L3.1
- new net: L3.2, R33.4
- no-connect marks 43 -> 40
Other:
- note added: "I_charge = 120mV / R -> 0.06ohm"
- note removed: "Detect if solar is above 10V -> it is Day prevent current flowing into disabled circuit due to low battery voltage prevent issues with reverse connected solar panel, e.g. Battery short due to shared ground"
- note removed: "Solar>~10V"
- moved on the sheet: D10, D11, ExtCharge1, IsDayBattery1, R78, R79, R9, U36

Commit message: layouted further
Parts:
- removed BatteryIn1, SolarIn1: TestPoint, symbol Connector:TestPoint
- removed D11: SS54, Diode_SMD:D_SMB-SMC_Universal_Handsoldering, symbol Device:D
- removed R8: 10k, Resistor_SMD:R_0603_1608Metric, symbol Device:R
- removed TP4: LED_+, TestPoint:TestPoint_THTPad_D2.0mm_Drill1.0mm, symbol Connector:TestPoint
- removed TP6: LED_-, TestPoint:TestPoint_THTPad_D2.0mm_Drill1.0mm, symbol Connector:TestPoint
- removed TP7: Feedback_LED, TestPoint:TestPoint_THTPad_D2.0mm_Drill1.0mm, symbol Connector:TestPoint
- added D11: LED, LED_SMD:LED_0603_1608Metric, symbol Device:LED
- added D4: 2A 25V, Diode_SMD:D_SMA, symbol Device:D
- added R26: 10k, Resistor_SMD:R_0603_1608Metric, symbol Device:R
- C75: footprint (none) -> Capacitor_SMD:C_1210_3225Metric
- F1, F3: footprint (none) -> Fuse:Fuseholder_Clip-5x20mm_Eaton_1A5601-01_Inline_P20.80x6.76mm_D1.70mm_Horizontal
- IsDayBattery1: footprint (none) -> TestPoint:TestPoint_Pad_2.0x2.0mm
- TP25, TP8: footprint TestPoint:TestPoint_THTPad_D2.0mm_Drill1.0mm -> TestPoint:TestPoint_Pad_2.0x2.0mm
- renumbered J1 to SolarIn2, J3 to battery1
Connections:
- net GND: now also D11.1 (K); no longer U36.2
- net at D1.2 (A): now also U36.1
- net Light_cool: now reaches C2.2, L1.1, U1.5 (SW)
- net Light+: now reaches C3.1, C4.1, C72.1, L1.2, LIGHT1.2 (Pin_2), R23.1
- net 3_3IN: now reaches C1.1, R3.2, U1.2 (EN), U1.3 (IN)
- net at D10.2 (A), ExtCharge1.2 (Pin_2): now also D4.2 (A)
- net Light_In: now reaches C1.1, R3.2, U1.2 (EN), U1.3 (IN)
- net 3_3V_cool: now reaches C2.2, L1.1, U1.5 (SW)
- new net: D11.2 (A), R26.1
- new net: R26.2, U36.2

Commit message: changes
Parts:
- removed C77: C_Polarized, Capacitor_THT:CP_Radial_D13.0mm_P5.00mm, symbol Device:C_Polarized
- removed D101: SS54, Diode_SMD:D_SMB-SMC_Universal_Handsoldering, symbol Device:D_Schottky
- removed D99: WS2812B, LED_SMD:LED_WS2812B_PLCC4_5.0x5.0mm_P3.2mm, symbol LED:WS2812B
- removed F1, F3: 4A, Fuse:Fuseholder_Clip-5x20mm_Eaton_1A5601-01_Inline_P20.80x6.76mm_D1.70mm_Horizontal, symbol Device:Fuse
- added C77: C, Capacitor_SMD:C_1206_3216Metric, symbol Device:C
- added C78: 100n, Capacitor_SMD:C_0603_1608Metric, symbol Device:C
- added C79, C9: 47uF 30v, Capacitor_THT:CP_Radial_D5.0mm_P2.00mm, symbol Device:C_Polarized
- added Q3: N-channel 30V 5A, Package_TO_SOT_SMD:SOT-23, symbol ESP32-DEVKITC-32D:SL2300
- added U34: LM74700, Package_TO_SOT_SMD:SOT-23-6, symbol Power_Management:LM74700
- C73: footprint Capacitor_SMD:C_1206_3216Metric -> Capacitor_SMD:C_0805_2012Metric
- C76: value C_Polarized -> 47uF 30v; footprint Capacitor_THT:CP_Radial_D13.0mm_P5.00mm -> Capacitor_THT:CP_Radial_D5.0mm_P2.00mm
- D100: footprint Diode_SMD:D_SMB-SMC_Universal_Handsoldering -> Diode_SMD:D_SMB
- I2C2, I2C3: footprint LED_SMD:LED_0805_2012Metric_Castellated -> LED_SMD:LED_0603_1608Metric
- L3: value L -> 47uH
- Q6: footprint Package_SO:SOP-8_3.9x4.9mm_P1.27mm -> board:4435
- R27: value R_MPPT_LOW -> 2.4K
- R33: footprint Resistor_SMD:R_Shunt_Vishay_WSK2512_6332Metric_T1.19mm -> board:R_Shunt_Vishay_WSK2512_6332Metric_T1.19mm
Connections:
- net 12V: now also battery1.2 (Pin_2), C79.1, Q3.3 (D), U34.4 (CATHODE)
- net GND: now also C77.2, C79.2, C9.2, U34.2 (GND)
- net S_VIN: now also C77.1, C9.1
- net at C75.1, C76.1: now also R33.4, C78.1, Q3.2 (S), U34.3 (EN), U34.6 (ANODE); no longer R33.1
- net at R30.1, U6.7 (BAT): now also R33.3; no longer R33.2
- net at U6.8 (CSP): now also R33.2; no longer R33.3
- net at Q6.1 (D): now also D100.1 (K), L3.1
- net at L3.2: now also R33.1; no longer R33.4
- new net: C78.2, U34.1 (VCAP)
- new net: Q3.1 (G), U34.5 (GATE)
Other:
- note added: "Ideal Protection Diode"
- note added: "MPPT 14.6V"
- moved on the sheet: C73, C74, C75, C76, D1, D100, D11, D98, IsDayBattery1, L3, Q6, R25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

Commit message: updated layout
Parts:
- removed I2C2: GREEN, LED_SMD:LED_0603_1608Metric, symbol Device:LED
- removed Q12: N-channel 30V 5A, Package_TO_SOT_SMD:SOT-23, symbol ESP32-DEVKITC-32D:SL2300
- removed Q_PWR5: P-channel 50v 4A, Package_TO_SOT_SMD:SOT-23, symbol Transistor_FET:BSS84
- removed R70, R74: 1k, Resistor_SMD:R_0603_1608Metric, symbol Device:R
- removed R72, R76: 10k, Resistor_SMD:R_0603_1608Metric, symbol Device:R
- added D13, D74, D75: BAT54S, Package_TO_SOT_SMD:SOT-23, symbol Diode:BAS40-04
- added J2: Conn_01x02_MountingPin, Connector_JST:JST_PH_B2B-PH-SM4-TB_1x02-1MP_P2.00mm_Vertical, symbol Connector_Generic_MountingPin:Conn_01x02_MountingPin
- added Q4: N-channel 30V 5A, Package_TO_SOT_SMD:SOT-23, symbol ESP32-DEVKITC-32D:SL2300
- added R29: 50, Resistor_SMD:R_0603_1608Metric, symbol Device:R
- added R8: 1k, Resistor_SMD:R_0603_1608Metric, symbol Device:R
- J2: value Conn_01x02_Male -> Conn_01x02_MountingPin; symbol Connector:Conn_01x02_Male -> Connector_Generic_MountingPin:Conn_01x02_MountingPin
- R18: value 270 -> 10k; LCSC_PART_NUMBER C17590 -> C212284
- R27: value 2.4K -> 2.491K
- R30: value R -> 34k
- R32: value R -> 2.491k
- renumbered IsDayBattery1 to IsDay1, R_MPPT_HIGH1 to R31
Connections:
- net 3_3V: now also I2C1.1 (Pin_1), R11.1, R12.1, D13.2, D74.2, D75.2, R29.2
- net GND: now also J2.MP (MountPin), J2.MP (MountPin), J2.MP (MountPin), J2.MP (MountPin), J2.MP (MountPin), J2.MP (MountPin), J2.MP (MountPin), J2.MP (MountPin), J2.MP (MountPin), J2.MP (MountPin), J2.MP (MountPin), J2.MP (MountPin), J2.MP (MountPin), J2.MP (MountPin), J2.MP (MountPin), J2.MP (MountPin), J2.MP (MountPin), J2.MP (MountPin), J2.MP (MountPin), J2.MP (MountPin), J2.MP (MountPin), J2.MP (MountPin), J2.MP (MountPin), J2.MP (MountPin), R18.2, D13.1, D74.1, D75.1, J2.MP (MountPin), Q4.2 (S)
- net SCL: now also D74.3
- net SDA: now also D13.3
- net ENABLE_TANK: now reaches U4.12 (IO27)
- net ENABLE_TANK: now also R8.2
- net TANK_SENSOR: now reaches U4.5 (SENSOR_VN)
- net TANK_SENSOR: now also D75.3, J2.2 (Pin_2), R29.1
- net 12V renamed VBAT
- net 5K_12V renamed 5K_VBAT
- removed net PWR_I2C: D24.3, I2C1.1 (Pin_1), R11.1, R12.1, R18.1
- new net: D24.3, J2.1 (Pin_1), Q4.3 (D)
- new net: Q4.1 (G), R18.1, R8.1
- no-connect marks 40 -> 64
Other:
- note added: "IsDay"
- note added: "MPPT 14.87V"
- note added: "Tank Sensor"
- note removed: "MPPT 14.6V"
- moved on the sheet: 1WIRE1, D3, I2C1, R1

Commit message: added batterymanagemt
Parts:
- removed D13, D74: BAT54S, Package_TO_SOT_SMD:SOT-23, symbol Diode:BAS40-04
- removed I2C1: Conn_01x04, Connector_JST:JST_EH_B4B-EH-A_1x04_P2.50mm_Vertical, symbol Connector_Generic:Conn_01x04
- added C80, C81, C82: 1uF, Capacitor_SMD:C_0603_1608Metric, symbol Device:C
- added C83, C84, C85: 100nF, Capacitor_SMD:C_0603_1608Metric, symbol Device:C
- added D5: WHITE, LED_SMD:LED_0603_1608Metric, symbol Device:LED
- added Q3: N-channel 30V 5A, Package_TO_SOT_SMD:SOT-23, symbol ESP32-DEVKITC-32D:SL2300
- added R35: 300k, Resistor_SMD:R_0603_1608Metric, symbol Device:R
- added R36: 15k, Resistor_SMD:R_0603_1608Metric, symbol Device:R
- added R38: R_Shunt, board:R_Shunt_Vishay_WSK2512_6332Metric_T1.19mm, symbol Device:R_Shunt
- added R42, R7: 1k, Resistor_SMD:R_0603_1608Metric, symbol Device:R
- added R43, R44: R, Resistor_SMD:R_0603_1608Metric, symbol Device:R
- added R8: 10k, Resistor_SMD:R_0603_1608Metric, symbol Device:R
- added U35: BQ34Z100PWR-G1, kicad-stuff:SOP65P640X120-14N, symbol BQ34Z100PWR-G1:BQ34Z100PWR-G1
Connections:
- net 3_3V: now also C81.1, R42.2, U35.5 (CE), U35.6 (REGIN)
- net GND: now also SolarIn2.1 (Pin_1), C80.2, C81.2, C82.2, C83.2, C84.2, R38.1, U35.8 (VSS); no longer SolarIn2.2 (Pin_2), battery1.1 (Pin_1)
- net SCL: now also U35.13 (P4/SCL)
- net SDA: now also U35.14 (P3/SDA)
- net S_VIN: now also D4.1 (K), SolarIn2.2 (Pin_2); no longer SolarIn2.1 (Pin_1)
- net VBAT: now also R35.1
- new net: C83.1, C85.2, R43.1, U35.9 (SRP)
- new net: D5.1 (K), Q3.3 (D)
- new net: D5.2 (A), R42.1
- new net: C82.1, R35.2, R36.1, U35.4 (BAT)
- new net: C84.1, C85.1, R44.1, U35.10 (SRN)
- new net: R38.2, R44.2
- new net: Q3.1 (G), R7.2, R8.1
- new net: C80.1, U35.7 (REG25)
- new net: R36.2, R38.4, battery1.1 (Pin_1)
- new net: Q3.2 (S), R8.2
- new net: R38.3, R43.2
- new net BAT_ALERT: U35.1 (P2)
- new net BAT_LED: R7.1, U35.3 (P1)
- no-connect marks 64 -> 68
Other:
- note added: "Is this even correct? check output type"
- note added: "check if values are already as expected if not Set internal temperature sensor set design capacity reset () check if values are correctly saved https://github.com/xkam1x/BQ34Z100G1/blob/master/README.md LiFePO4 RELAX? usefull commands AvailableEnergy() AveragePower() StateOfHealth() ChargeCurrent()"
- moved on the sheet: battery1
