File: board/PlantCtrlESP32.kicad_sch (KiCad schematic)
At the start: 419 parts, among them J2 Conn_01x02_MountingPin, J2 Conn_01x03_Female, J2 Conn_01x07, Q2 N-channel 30V 5A, Q3 N-channel 30V 5A, Q4 N-channel 30V 5A, Q6 4435, U1 74HC595, U1 AP63200, U1 AP63203, U1 TLC555xP, U2 74HC595, U34 LM74700, U35 BQ34Z100PWR-G1, U36 PC817, U4 ESP32-WROOM-32D, U6 CN3795

Commit message: added bettry manager
Parts:
- removed R7: 1k, Resistor_SMD:R_0603_1608Metric, symbol Device:R
- removed R8: 10k, Resistor_SMD:R_0603_1608Metric, symbol Device:R
- added D5: RED, LED_SMD:LED_0603_1608Metric, symbol Device:LED
- added Q3: N-channel 30V 5A, Package_TO_SOT_SMD:SOT-23, symbol ESP32-DEVKITC-32D:SL2300
- added R39: 1k, Resistor_SMD:R_0603_1608Metric, symbol Device:R
- added R40: 10k, Resistor_SMD:R_0603_1608Metric, symbol Device:R
Connections:
- net 3_3V: now also R39.2
- net BAT_ALERT: now also Q3.1 (G), R40.2
- net BAT_LED: now also Q3.1 (G)
- net GND: now also Q3.2 (S), RV1.1, Q3.2 (S); no longer RV1.3
- net at R24.2: now also RV1.3; no longer RV1.1
- net REG25: now reaches C80.1, U35.7 (REG25)
- net REG25: now also R40.1
- new net: D5.1 (K), Q3.3 (D)
- new net: D5.2 (A), R39.1
- no-connect marks 68 -> 71
Other:
- note added: "free"
- note removed: "Is this even correct? check output type"
- moved on the sheet: C80, D5, Q3, R12, R42

Commit message: finalize
Parts:
- C75: value C -> 25V 10uF; footprint Capacitor_SMD:C_1210_3225Metric -> Capacitor_SMD:C_1206_3216Metric
- C77: value C -> 25V 10uF
- D10, D11, D2, D5, D98, I2C3, P_FAULT1, P_FAULT2, P_FAULT3, P_FAULT4, P_FAULT5, P_FAULT6, P_FAULT7, P_FAULT8, SD1, SD25, SD26, SD27, SD28, SD29, SD30, SD31, SD32, SD33, SD34, SD35, SD36, SD37, SD38, SD39, SD40, SD41, SD42, SD43, SD44, SD45, SD46, SD47: footprint LED_SMD:LED_0603_1608Metric -> LED_SMD:LED_0805_2012Metric
Other:
- note added: "Battery Management"
- moved on the sheet: C80, C81, C82, C83, C84, C85, D5, Q3, R35, R36, R38, R39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

Commit message: finalize layout for comparator
Parts:
- removed D1: 7v zehner, Diode_SMD:D_SOD-123, symbol Device:D_Zener
- removed R78: 1k, Resistor_SMD:R_0603_1608Metric, symbol Device:R
- removed R79: 10k, Resistor_SMD:R_0603_1608Metric, symbol Device:R
- removed U36: PC817, Package_DIP:DIP-4_W7.62mm, symbol Isolator:PC817
- added C88: 100pf, Capacitor_SMD:C_0603_1608Metric, symbol Device:C
- added D16: BAT54S, Package_TO_SOT_SMD:SOT-23, symbol Diode:BAS40-04
- added R54, R57, R60, R66: 10k, Resistor_SMD:R_0603_1608Metric, symbol Device:R
- added R63: 1k, Resistor_SMD:R_0603_1608Metric, symbol Device:R
- added U36: GS331, Package_TO_SOT_SMD:SOT-23-5, symbol Comparator:LM397
- R26: value 10k -> 50k
Connections:
- net 3_3V: now also D16.2, R57.1, U36.5 (V+)
- net BAT_LED: now also R66.1
- net GND: now also C88.2, R54.2, R60.2, R66.2, U36.2 (V-)
- net IsDay: now also R63.1, U36.4
- net S_VIN: now also R26.1
- net EXT_3V3: now reaches U4.8 (IO32)
- net EXT_12V: now reaches U4.9 (IO33)
- net at D11.2 (A): now also R63.2; no longer R26.1
- net at R26.2: now also C88.1, D16.1, R54.1
- net CentralPump: no longer names the net of D5.1 (K), D6.3, PUMP9.1 (Pin_1), Q3.3 (D)
- new net: D16.3, U36.3 (+)
- new net: R57.2, R60.1, U36.1 (-)
- no-connect marks 71 -> 69
Other:
- note added: "FreeAnyStuff"
- note removed: "CentralPump"
- moved on the sheet: D11, IsDay1

Commit message: fix reverse protection diodes
Connections:
- net 3_3V: now also D23.2, D24.2, D25.2, D26.2; no longer D23.1, D24.1, D25.1, D26.1
- net GND: now also D23.1, D24.1, D25.1, D26.1; no longer D23.2, D24.2, D25.2, D26.2
Changed lines of the file:
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@@
     )
   )
-  (global_label "GND" (shape input) (at 483.108 322.834 180) (fields_autoplaced)
-    (effects (font (size 1.27 1.27)) (justify right))
-    (property "Intersheetrefs" "${INTERSHEET_REFS}" (at 476.9859 322.834 0)
-      (effects (font (size 1.27 1.27)) (justify right) hide)
+  (global_label "GND" (shape input) (at 498.348 322.834 0) (fields_autoplaced)
+    (effects (font (size 1.27 1.27)) (justify left))
+    (property "Intersheetrefs" "${INTERSHEET_REFS}" (at 504.5495 322.834 0)
+      (effects (font (size 1.27 1.27)) (justify left) hide)
     )
   )
@@
     )
   )
-  (global_label "3_3V" (shape input) (at 498.348 322.834 0) (fields_autoplaced)
-    (effects (font (size 1.27 1.27)) (justify left))
-    (property "Intersheetrefs" "${INTERSHEET_REFS}" (at 505.0748 322.834 0)
-      (effects (font (size 1.27 1.27)) (justify left) hide)
+  (global_label "3_3V" (shape input) (at 483.108 322.834 180) (fields_autoplaced)
+    (effects (font (size 1.27 1.27)) (justify right))
+    (property "Intersheetrefs" "${INTERSHEET_REFS}" (at 476.3018 322.834 0)
+      (effects (font (size 1.27 1.27)) (justify right) hide)
     )
   )
@@
     )
   )
-  (global_label "3_3V" (shape input) (at 480.568 283.464 180) (fields_autoplaced)
-    (effects (font (size 1.27 1.27)) (justify right))
-    (property "Intersheetrefs" "${INTERSHEET_REFS}" (at 473.8412 283.464 0)
-      (effects (font (size 1.27 1.27)) (justify right) hide)
+  (global_label "3_3V" (shape input) (at 495.808 283.464 0) (fields_autoplaced)
+    (effects (font (size 1.27 1.27)) (justify left))
+    (property "Intersheetrefs" "${INTERSHEET_REFS}" (at 502.6142 283.464 0)
+      (effects (font (size 1.27 1.27)) (justify left) hide)
     )
   )
@@
     )
   )
-  (global_label "GND" (shape input) (at 511.048 322.834 180) (fields_autoplaced)
-    (effects (font (size 1.27 1.27)) (justify right))
-    (property "Intersheetrefs" "${INTERSHEET_REFS}" (at 504.9259 322.834 0)
-      (effects (font (size 1.27 1.27)) (justify right) hide)
+  (global_label "GND" (shape input) (at 526.288 322.834 0) (fields_autoplaced)
+    (effects (font (size 1.27 1.27)) (justify left))
+    (property "Intersheetrefs" "${INTERSHEET_REFS}" (at 532.4895 322.834 0)
+      (effects (font (size 1.27 1.27)) (justify left) hide)
     )
   )
@@
     )
   )
-  (global_label "3_3V" (shape input) (at 509.778 283.464 180) (fields_autoplaced)
-    (effects (font (size 1.27 1.27)) (justify right))
-    (property "Intersheetrefs" "${INTERSHEET_REFS}" (at 503.0512 283.464 0)
-      (effects (font (size 1.27 1.27)) (justify right) hide)
+  (global_label "3_3V" (shape input) (at 525.018 283.464 0) (fields_autoplaced)
+    (effects (font (size 1.27 1.27)) (justify left))
+    (property "Intersheetrefs" "${INTERSHEET_REFS}" (at 531.8242 283.464 0)
+      (effects (font (size 1.27 1.27)) (justify left) hide)
     )
   )
@@
     )
   )
-  (global_label "GND" (shape input) (at 525.018 283.464 0) (fields_autoplaced)
-    (effects (font (size 1.27 1.27)) (justify left))
-    (property "Intersheetrefs" "${INTERSHEET_REFS}" (at 531.1401 283.464 0)
-      (effects (font (size 1.27 1.27)) (justify left) hide)
+  (global_label "GND" (shape input) (at 509.778 283.464 180) (fields_autoplaced)
+    (effects (font (size 1.27 1.27)) (justify right))
+    (property "Intersheetrefs" "${INTERSHEET_REFS}" (at 503.5765 283.464 0)
+      (effects (font (size 1.27 1.27)) (justify right) hide)
     )
   )
@@
     )
   )
-  (global_label "GND" (shape input) (at 495.808 283.464 0) (fields_autoplaced)
-    (effects (font (size 1.27 1.27)) (justify left))
-    (property "Intersheetrefs" "${INTERSHEET_REFS}" (at 501.9301 283.464 0)
-      (effects (font (size 1.27 1.27)) (justify left) hide)
+  (global_label "GND" (shape input) (at 480.568 283.464 180) (fields_autoplaced)
+    (effects (font (size 1.27 1.27)) (justify right))
+    (property "Intersheetrefs" "${INTERSHEET_REFS}" (at 474.3665 283.464 0)
+      (effects (font (size 1.27 1.27)) (justify right) hide)
     )
   )
@@
     )
   )
-  (global_label "3_3V" (shape input) (at 526.288 322.834 0) (fields_autoplaced)
-    (effects (font (size 1.27 1.27)) (justify left))
-    (property "Intersheetrefs" "${INTERSHEET_REFS}" (at 533.0148 322.834 0)
-      (effects (font (size 1.27 1.27)) (justify left) hide)
-    )
-  )
+  (global_label "3_3V" (shape input) (at 511.048 322.834 180) (fields_autoplaced)
+    (effects (font (size 1.27 1.27)) (justify right))
+    (property "Intersheetrefs" "${INTERSHEET_REFS}" (at 504.2418 322.834 0)
+      (effects (font (size 1.27 1.27)) (justify right) hide)
+    )
+  )

Commit message: fix for reset of shift register
Connections:
- net 3_3V: now also U1.10 (~{SRCLR}), U1.10 (~{SRCLR}), U2.10 (~{SRCLR}), U2.10 (~{SRCLR}), U2.10 (~{SRCLR})
- no-connect marks 69 -> 64
Changed lines of the file:
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@@
   (no_connect (at 409.448 183.388))
   (no_connect (at 634.238 149.098))
-  (no_connect (at 225.298 313.944))
   (no_connect (at 547.878 183.388))
   (no_connect (at 404.368 149.098))
@@
   (no_connect (at 107.696 97.282))
   (no_connect (at 107.696 87.122))
-  (no_connect (at 326.898 313.944))
   (no_connect (at 77.216 112.522))
   (no_connect (at 495.808 149.098))
@@
   (no_connect (at 727.456 43.434))
   (no_connect (at 549.656 77.724))
-  (no_connect (at 428.498 313.944))
   (no_connect (at 409.956 77.724))
   (no_connect (at 450.596 43.434))
@@
   (no_connect (at 455.168 183.388))
   (no_connect (at 364.236 77.724))
-  (no_connect (at 377.698 313.944))
   (no_connect (at 311.658 149.098))
   (no_connect (at 497.586 43.434))
@@
   (no_connect (at 568.325 357.251))
   (no_connect (at 589.026 43.434))
-  (no_connect (at 276.098 313.944))
   (no_connect (at 732.536 77.724))
   (no_connect (at 77.216 109.982))
@@
     )
   )
+  (global_label "3_3V" (shape input) (at 276.098 313.944 270) (fields_autoplaced)
+    (effects (font (size 1.27 1.27)) (justify right))
+    (property "Intersheetrefs" "${INTERSHEET_REFS}" (at 276.098 320.7502 90)
+      (effects (font (size 1.27 1.27)) (justify right) hide)
+    )
+  )
   (global_label "3_3V" (shape input) (at 603.758 184.658 0) (fields_autoplaced)
     (effects (font (size 1.27 1.27)) (justify left))
@@
     )
   )
+  (global_label "3_3V" (shape input) (at 428.498 313.944 270) (fields_autoplaced)
+    (effects (font (size 1.27 1.27)) (justify right))
+    (property "Intersheetrefs" "${INTERSHEET_REFS}" (at 428.498 320.7502 90)
+      (effects (font (size 1.27 1.27)) (justify right) hide)
+    )
+  )
   (global_label "EXT_12V" (shape input) (at 107.696 127.762 0) (fields_autoplaced)
     (effects (font (size 1.27 1.27)) (justify left))
@@
     )
   )
+  (global_label "3_3V" (shape input) (at 377.698 313.944 270) (fields_autoplaced)
+    (effects (font (size 1.27 1.27)) (justify right))
+    (property "Intersheetrefs" "${INTERSHEET_REFS}" (at 377.698 320.7502 90)
+      (effects (font (size 1.27 1.27)) (justify right) hide)
+    )
+  )
   (global_label "3_3V" (shape input) (at 603.885 272.923 90) (fields_autoplaced)
     (effects (font (size 1.27 1.27)) (justify left))
@@
     )
   )
+  (global_label "3_3V" (shape input) (at 326.898 313.944 270) (fields_autoplaced)
+    (effects (font (size 1.27 1.27)) (justify right))
+    (property "Intersheetrefs" "${INTERSHEET_REFS}" (at 326.898 320.7502 90)
+      (effects (font (size 1.27 1.27)) (justify right) hide)
+    )
+  )
   (global_label "GND" (shape input) (at 498.348 144.018 180) (fields_autoplaced)
     (effects (font (size 1.27 1.27)) (justify right))
@@
     )
   )
+  (global_label "3_3V" (shape input) (at 225.298 313.944 270) (fields_autoplaced)
+    (effects (font (size 1.27 1.27)) (justify right))
+    (property "Intersheetrefs" "${INTERSHEET_REFS}" (at 225.298 320.7502 90)
+      (effects (font (size 1.27 1.27)) (justify right) hide)
+    )
+  )

Commit message: set mppt output voltage to be less agressive
Parts:
- R30: value 34k -> 30k
Changed lines of the file:
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@@
       (effects (font (size 1.27 1.27)) (justify left))
     )
-    (property "Value" "34k" (at 435.61 615.95 0)
+    (property "Value" "30k" (at 435.61 615.95 0)
       (effects (font (size 1.27 1.27)) (justify left))
     )

Commit message: add i2c initial and pull configs
Parts:
- added R45: 1k ? unclear if required, Resistor_SMD:R_0603_1608Metric, symbol Device:R
Connections:
- net IsDay: now also R45.2; no longer U4.10 (IO25)
- new net: R45.1, U4.10 (IO25)
Changed lines of the file:
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@@
     )
   )
-  (global_label "IsDay" (shape input) (at 107.696 117.602 0) (fields_autoplaced)
+  (global_label "IsDay" (shape input) (at 115.316 117.602 0) (fields_autoplaced)
     (effects (font (size 1.27 1.27)) (justify left))
-    (property "Intersheetrefs" "${INTERSHEET_REFS}" (at 114.9671 117.602 0)
+    (property "Intersheetrefs" "${INTERSHEET_REFS}" (at 122.5871 117.602 0)
       (effects (font (size 1.27 1.27)) (justify left) hide)
     )
@@
         )
       )
+    )
+  )
+  (symbol (lib_id "Device:R") (at 111.506 117.602 90) (unit 1)
+    (in_bom yes) (on_board yes) (dnp no)
+    (property "Reference" "R45" (at 111.506 112.522 90)
+      (effects (font (size 1.27 1.27)))
+    )
+    (property "Value" "1k ? unclear if required" (at 134.874 115.062 90)
+      (effects (font (size 1.27 1.27)))
+    )
+    (property "Footprint" "Resistor_SMD:R_0603_1608Metric" (at 111.506 119.38 90)
+      (effects (font (size 1.27 1.27)) hide)
+    )
+    (property "Datasheet" "~" (at 111.506 117.602 0)
+      (effects (font (size 1.27 1.27)) hide)
+    )
+    (pin "1")
+    (pin "2")
+    (instances
+      (project "PlantCtrlESP32"
+        (path "/c26e8d55-0b6e-4c4e-b7c8-b1fed973201c"
+          (reference "R45") (unit 1)
+        )
+      )

Commit message: fix for bq34z100 led mode, added i2c header
Parts:
- added J1: Conn_01x03_Female, Connector_PinHeader_2.54mm:PinHeader_1x03_P2.54mm_Vertical, symbol Connector:Conn_01x03_Male
Connections:
- net 3_3V: now also U35.2 (VEN)
- net GND: now also J1.1 (Pin_1)
- net SCL: now also J1.2 (Pin_2)
- net SDA: now also J1.3 (Pin_3)
- no-connect marks 64 -> 63
Changed lines of the file:
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@@
   (no_connect (at 455.676 77.724))
   (no_connect (at 544.576 43.434))
-  (no_connect (at 603.885 377.571))
   (no_connect (at 733.298 183.388))
   (no_connect (at 542.798 149.098))
@@
     (stroke (width 0) (type default))
   )
+  (wire (pts (xy 603.885 377.571) (xy 606.933 377.571))
+    (stroke (width 0) (type default))
+  )
   (wire (pts (xy 518.668 311.404) (xy 518.668 317.754))
     (stroke (width 0) (type default))
@@
     )
   )
+  (global_label "3_3V" (shape input) (at 606.933 377.571 0) (fields_autoplaced)
+    (effects (font (size 1.27 1.27)) (justify left))
+    (property "Intersheetrefs" "${INTERSHEET_REFS}" (at 613.7392 377.571 0)
+      (effects (font (size 1.27 1.27)) (justify left) hide)
+    )
+  )
   (global_label "GND" (shape input) (at 167.386 92.202 0) (fields_autoplaced)
     (effects (font (size 1.27 1.27)) (justify left))
@@
     )
   )
+  (global_label "GND" (shape input) (at 569.595 314.96 0) (fields_autoplaced)
+    (effects (font (size 1.27 1.27)) (justify left))
+    (property "Intersheetrefs" "${INTERSHEET_REFS}" (at 575.7965 314.96 0)
+      (effects (font (size 1.27 1.27)) (justify left) hide)
+    )
+  )
   (global_label "GND" (shape input) (at 498.348 144.018 180) (fields_autoplaced)
     (effects (font (size 1.27 1.27)) (justify right))
@@
     )
   )
+  (global_label "SDA" (shape input) (at 569.595 320.04 0) (fields_autoplaced)
+    (effects (font (size 1.27 1.27)) (justify left))
+    (property "Intersheetrefs" "${INTERSHEET_REFS}" (at 575.4147 320.04 0)
+      (effects (font (size 1.27 1.27)) (justify left) hide)
+    )
+  )
+  (global_label "SCL" (shape input) (at 569.595 317.5 0) (fields_autoplaced)
+    (effects (font (size 1.27 1.27)) (justify left))
+    (property "Intersheetrefs" "${INTERSHEET_REFS}" (at 575.4336 317.5 0)
+      (effects (font (size 1.27 1.27)) (justify left) hide)
+    )
+  )
   (global_label "SDA" (shape input) (at 603.885 357.251 0) (fields_autoplaced)
     (effects (font (size 1.27 1.27)) (justify left))
@@
         )
       )
+    )
+  )
+  (symbol (lib_id "Connector:Conn_01x03_Male") (at 564.515 317.5 0) (unit 1)
+    (in_bom yes) (on_board yes) (dnp no)
+    (property "Reference" "J1" (at 560.451 318.77 0)
+      (effects (font (size 1.27 1.27)) (justify left))
+    )
+    (property "Value" "Conn_01x03_Female" (at 552.323 321.818 0)
+      (effects (font (size 1.27 1.27)) (justify left))
+    )
+    (property "Footprint" "Connector_PinHeader_2.54mm:PinHeader_1x03_P2.54mm_Vertical" (at 564.515 317.5 0)
+      (effects (font (size 1.27 1.27)) hide)
+    )
+    (property "Datasheet" "~" (at 564.515 317.5 0)
+      (effects (font (size 1.27 1.27)) hide)
+    )
+    (pin "1")
+    (pin "2")
+    (pin "3")
+    (instances
+      (project "PlantCtrlESP32"
+        (path "/c26e8d55-0b6e-4c4e-b7c8-b1fed973201c"
+          (reference "J1") (unit 1)
+        )
+      )
